Commit message: first complete version of s5fs_gripper with mimics

File: s5fs_gripper/description/urdf/s5fs.urdf (robot description, URDF)
Before this commit: robot s5fs, 15 links, 14 joints
Links:
- added link e; visual cylinder length=0.0215 radius=0.001
- added link e1; visual cylinder length=0.0375 radius=0.001
- added link e2; visual cylinder length=0.0175 radius=0.001
- added link e3; visual cylinder length=0.03 radius=0.001
- added link e4; visual cylinder length=0.026 radius=0.001
- added link e5; visual cylinder length=0.0355 radius=0.001
- added link i; visual cylinder length=0.04454 radius=0.001
- added link j; visual cylinder length=0.05004 radius=0.001
- added link m; visual cylinder length=0.022 radius=0.001
- added link n; visual cylinder length=0.032 radius=0.001
- added link q; visual cylinder length=0.015 radius=0.001
- added link r; visual cylinder length=0.015 radius=0.001
- added link virtual_i; visual cylinder length=0 radius=0
- added link virtual_j; visual cylinder length=0 radius=0
- link a: geometry visual cylinder length=0.0485 radius=0.001
- link b: geometry visual cylinder length=0.030 radius=0.001
- link base_link: geometry visual box size=0.0353 0.02626 0.010
- link c: geometry visual cylinder length=0.020 radius=0.001
- link d: geometry visual cylinder length=0.110 radius=0.001
- link d2: geometry visual cylinder length=0.0275 radius=0.001
- link h: geometry visual cylinder length=0.025 radius=0.001
- link k: geometry visual cylinder length=0.05004 radius=0.001
- link l: geometry visual cylinder length=0.04804 radius=0.001
- link o: geometry visual cylinder length=0.032 radius=0.001
- link p: geometry visual cylinder length=0.026 radius=0.001
- link s: geometry visual cylinder length=0.015 radius=0.001
- link t: geometry visual cylinder length=0.015 radius=0.001
- link virtual_l: geometry visual cylinder length=0 radius=0
- link z: geometry visual cylinder length=0.04596 radius=0.001
Joints:
- removed joint j1
- removed joint j10
- removed joint j11
- removed joint j2
- removed joint j6a
- removed joint j6b
- removed joint j7
- added joint f4: type fixed, parent base_link, child e1, origin xyz=0 0 0 rpy=0 0 0
- added joint f5: type fixed, parent e2, child e3, origin xyz=0 0 0 rpy=0 0 0
- added joint f6: type fixed, parent e3, child e, origin xyz=0 0 0 rpy=0 0 0
- added joint f7: type fixed, parent e, child e4, origin xyz=0 0 0 rpy=0 0 0
- added joint f8: type fixed, parent e, child e5, origin xyz=0 0 0 rpy=0 0 0
- added joint j10_forefinger2: type revolute, parent l, child p, origin xyz=0 0 0.04804 rpy=0 0 0, axis -1 0 0, limit lower=0 upper=1.334 effort=1000.0 velocity=1
- added joint j11_middlefinger2: type revolute, parent k, child o, origin xyz=0 0 0.05004 rpy=0 0 0, axis -1 0 0, limit lower=0 upper=1.334 effort=1000.0 velocity=1
- added joint j12: type revolute, parent j, child n, origin xyz=0 0 0.05004 rpy=0 0 0, axis -1 0 0, limit lower=0 upper=1.334 effort=1000.0 velocity=1, mimic joint=j8a_ringfinger multiplier=1.3588 offset=0
- added joint j13: type revolute, parent i, child m, origin xyz=0 0 0.04454 rpy=0 0 0, axis -1 0 0, limit lower=0 upper=1.334 effort=1000.0 velocity=1, mimic joint=j9a_littlefinger multiplier=1.35880 offset=0
- added joint j16: type revolute, parent n, child r, origin xyz=0 0 0.032 rpy=0 0 0, axis -1 0 0, limit lower=0 upper=1.395 effort=1000.0 velocity=1, mimic joint=j8a_ringfinger multiplier=1.42093 offset=0
- added joint j17: type revolute, parent m, child q, origin xyz=0 0 0.022 rpy=0 0 0, axis -1 0 0, limit lower=0 upper=1.3971 effort=1000.0 velocity=1, mimic joint=j9a_littlefinger multiplier=1.42307 offset=0
- added joint j1_wrist: type revolute, parent base_link, child z, origin xyz=-0.01690 0.02626 0 rpy=0 0.2618 1.571, axis 0 0 -1, limit lower=0.0 upper=0.9879 effort=1000.0 velocity=1
- added joint j2_thumb: type revolute, parent z, child a, origin xyz=0 0 0.04596 rpy=0 0 0, axis 1 0 0, limit lower=0.0 upper=0.9704 effort=1000.0 velocity=1
- added joint j5: type revolute, parent e1, child e2, origin xyz=0.01840 0 0.0375 rpy=0 0 0, axis 0 0 1, limit lower=0.0 upper=0.98786 effort=1000.0 velocity=1, mimic joint=j1_wrist multiplier=1 offset=0
- added joint j6a_forefinger1: type revolute, parent d2, child virtual_l, origin xyz=-0.025 0 0.110 rpy=0 0 0, axis -1 0 0, limit lower=0.0 upper=0.79849 effort=1000.0 velocity=1
- added joint j6b_spread: type revolute, parent virtual_l, child l, origin xyz=0 0 0 rpy=0 0 0, axis 0 -1 0, limit lower=0.0 upper=0.28833 effort=1000.0 velocity=1
- added joint j7_middlefinger1: type revolute, parent d, child k, origin xyz=0 0 0.110 rpy=0 0 0, axis -1 0 0, limit lower=0.0 upper=0.79849 effort=1000.0 velocity=1
- added joint j8a_ringfinger: type revolute, parent e5, child virtual_j, origin xyz=0 0 0.0655 rpy=0 0 0, axis -1 0 0, limit lower=0.0 upper=0.98175 effort=1000.0 velocity=1
- added joint j8b: type revolute, parent virtual_j, child j, origin xyz=0.00675 0 0 rpy=0 0 0, axis 0 1 0, limit lower=0.0 upper=0.28833 effort=1000.0 velocity=1, mimic joint=j6b_spread multiplier=1 offset=0
- added joint j9a_littlefinger: type revolute, parent e4, child virtual_i, origin xyz=0 0 0.056 rpy=0 0 0, axis -1 0 0, limit lower=0.0 upper=0.98175 effort=1000.0 velocity=1
- added joint j9b: type revolute, parent virtual_i, child i, origin xyz=0.02825 0 0 rpy=0 0 0, axis 0 1 0, limit lower=0.0 upper=0.5829 effort=1000.0 velocity=1, mimic joint=j6b_spread multiplier=2.02164 offset=0
- joint j14: mimic (none) -> joint=j10_forefinger2 multiplier=1.0450 offset=0; origin xyz=0 0 0.26 rpy=0 0 0 -> xyz=0 0 0.026 rpy=0 0 0
- joint j15: mimic (none) -> joint=j11_middlefinger2 multiplier=1.000 offset=0; origin xyz=0 0 0.32 rpy=0 0 0 -> xyz=0 0 0.032 rpy=0 0 0
- joint j3: mimic (none) -> joint=j2_thumb multiplier=1.01511 offset=0; origin xyz=0 0 0.4596 rpy=0 0 0 -> xyz=0 0 0.0485 rpy=0 0 0
- joint j4: mimic (none) -> joint=j2_thumb multiplier=1.44889 offset=0; origin xyz=0 0 0.3 rpy=0 0 0 -> xyz=0 0 0.030 rpy=0 0 0
