Commit message: adapted urdf to schunk naming conventions

File: s5fh_gripper/description/urdf/s5fs.urdf.xacro (robot description, xacro)
@@ -275,6 +275,13 @@
         </visual>
     </link>
+   <joint name="Thumb_Flexion" type="revolute">
+        <parent link="z" />
+        <child link="a" />
+        <limit effort="1000.0" lower="0.0" upper="0.9704" velocity="1" />
+        <origin xyz="0 0 0.04596" rpy="0 0 0" />
+        <axis xyz="${orientation*(1)} 0 0" />
+    </joint>
     <!-- BASE_LINE JOINTS -->
-    <joint name="j1_wrist" type="revolute">
+    <joint name="Thumb_Opposition" type="revolute">
         <parent link="base_link" />
         <child link="z" />
@@ -284,11 +291,4 @@
     </joint>
     <!-- JOINT NOT FOR BASE_LINE. BUT WRITTEN DOWN HERE FOR BETTER UX -->
-    <joint name="j6b_spread" type="revolute">
-        <parent link="virtual_l" />
-        <child link="l" />
-        <limit effort="1000.0" lower="0.0" upper="0.28833" velocity="1" />
-        <origin xyz="0 0 0" rpy="0 0 0" />
-        <axis xyz="0 ${orientation*(-1)} 0" />
-    </joint>
     <joint name="f1" type="fixed">
         <parent link="base_link" />
@@ -317,5 +317,5 @@
         <origin xyz="${orientation*(0.01840)} 0 0.0375" rpy="0 0 0" />
         <axis xyz="0 0 ${orientation*(1)}" />
-        <mimic joint="j1_wrist" multiplier="1" offset="0" />
+        <mimic joint="Thumb_Opposition" multiplier="1" offset="0" />
     </joint>
     <joint name="f5" type="fixed">
@@ -340,11 +340,4 @@
     </joint>
     <!-- THUMB JOINTS -->
-    <joint name="j2_thumb" type="revolute">
-        <parent link="z" />
-        <child link="a" />
-        <limit effort="1000.0" lower="0.0" upper="0.9704" velocity="1" />
-        <origin xyz="0 0 0.04596" rpy="0 0 0" />
-        <axis xyz="${orientation*(1)} 0 0" />
-    </joint>
     <joint name="j3" type="revolute">
         <parent link="a" />
@@ -353,5 +346,5 @@
         <origin xyz="0 0 0.0485" rpy="0 0 0" />
         <axis xyz="${orientation*(1)} 0 0" />
-        <mimic joint="j2_thumb" multiplier="1.01511" offset="0" />
+        <mimic joint="Thumb_Flexion" multiplier="1.01511" offset="0" />
     </joint>
     <joint name="j4" type="revolute">
@@ -361,8 +354,15 @@
         <origin xyz="0 0 0.030" rpy="0 0 0" />
         <axis xyz="${orientation*(1)} 0 0" />
-        <mimic joint="j2_thumb" multiplier="1.44889" offset="0" />
+        <mimic joint="Thumb_Flexion" multiplier="1.44889" offset="0" />
     </joint>
     <!-- FOREFINGER JOINTS -->
-    <joint name="j6a_forefinger1" type="revolute">
+    <joint name="Index_Finger_Distal" type="revolute">
+        <parent link="l" />
+        <child link="p" />
+        <limit effort="1000.0" lower="0" upper="1.334" velocity="1" />
+        <origin xyz="0 0 0.04804" rpy="0 0 0" />
+        <axis xyz="-1 0 0" />
+    </joint>
+    <joint name="Index_Finger_Proximal" type="revolute">
         <parent link="d2" />
         <child link="virtual_l" />
@@ -371,13 +371,6 @@
         <axis xyz="-1 0 0" />
     </joint>
-    <!-- JOINT j6b_spread in BASE_LINE section for better UX -->
-    <joint name="j10_forefinger2" type="revolute">
-        <parent link="l" />
-        <child link="p" />
-        <limit effort="1000.0" lower="0" upper="1.334" velocity="1" />
-        <origin xyz="0 0 0.04804" rpy="0 0 0" />
-        <axis xyz="-1 0 0" />
-    </joint>
-    <joint name="j14" type="revolute">
+    <!-- JOINT Finger_Spread in BASE_LINE section for better UX -->
+     <joint name="j14" type="revolute">
         <parent link="p" />
         <child link="t" />
@@ -385,8 +378,15 @@
         <origin xyz="0 0 0.026" rpy="0 0 0" />
         <axis xyz="-1 0 0" />
-        <mimic joint="j10_forefinger2" multiplier="1.0450" offset="0" />
+        <mimic joint="Index_Finger_Distal" multiplier="1.0450" offset="0" />
     </joint>
     <!-- MIDDLE FINGER JOINTS -->
-    <joint name="j7_middlefinger1" type="revolute">
+    <joint name="Middle_Finger_Distal" type="revolute">
+        <parent link="k" />
+        <child link="o" />
+        <limit effort="1000.0" lower="0" upper="1.334" velocity="1" />
+        <origin xyz="0 0 0.05004" rpy="0 0 0" />
+        <axis xyz="-1 0 0" />
+    </joint>
+    <joint name="Middle_Finger_Proximal" type="revolute">
         <parent link="d" />
         <child link="k" />
@@ -395,12 +395,5 @@
         <axis xyz="-1 0 0" />
     </joint>
-    <joint name="j11_middlefinger2" type="revolute">
-        <parent link="k" />
-        <child link="o" />
-        <limit effort="1000.0" lower="0" upper="1.334" velocity="1" />
-        <origin xyz="0 0 0.05004" rpy="0 0 0" />
-        <axis xyz="-1 0 0" />
-    </joint>
-    <joint name="j15" type="revolute">
+     <joint name="j15" type="revolute">
         <parent link="o" />
         <child link="s" />
@@ -408,8 +401,8 @@
         <origin xyz="0 0 0.032" rpy="0 0 0" />
         <axis xyz="-1 0 0" />
-        <mimic joint="j11_middlefinger2" multiplier="1.000" offset="0" />
+        <mimic joint="Middle_Finger_Distal" multiplier="1.000" offset="0" />
     </joint>
     <!-- RING FINGER JOINTS -->
-    <joint name="j8a_ringfinger" type="revolute">
+    <joint name="Ring_Finger" type="revolute">
         <parent link="e5" />
         <child link="virtual_j" />
@@ -424,5 +417,5 @@
         <origin xyz="${orientation*(0.00675)} 0 0" rpy="0 0 0" />
         <axis xyz="0 ${orientation*(1)} 0" />
-        <mimic joint="j6b_spread" multiplier="1" offset="0" />
+        <mimic joint="Finger_Spread" multiplier="1" offset="0" />
     </joint>
     <joint name="j12" type="revolute">
@@ -432,5 +425,5 @@
         <origin xyz="0 0 0.05004" rpy="0 0 0" />
         <axis xyz="-1 0 0" />
-        <mimic joint="j8a_ringfinger" multiplier="1.3588" offset="0" />
+        <mimic joint="Ring_Finger" multiplier="1.3588" offset="0" />
     </joint>
     <joint name="j16" type="revolute">
@@ -440,8 +433,8 @@
         <origin xyz="0 0 0.032" rpy="0 0 0" />
         <axis xyz="-1 0 0" />
-        <mimic joint="j8a_ringfinger" multiplier="1.42093" offset="0" />
+        <mimic joint="Ring_Finger" multiplier="1.42093" offset="0" />
     </joint>
     <!-- LITTLE FINGER JOINTS -->
-    <joint name="j9a_littlefinger" type="revolute">
+    <joint name="Pinky" type="revolute">
         <parent link="e4" />
         <child link="virtual_i" />
@@ -456,5 +449,5 @@
         <origin xyz="${orientation*(0.02825)} 0 0" rpy="0 0 0" />
         <axis xyz="0 ${orientation*(1)} 0" />
-        <mimic joint="j6b_spread" multiplier="2.02164" offset="0" />
+        <mimic joint="Finger_Spread" multiplier="2.02164" offset="0" />
     </joint>
     <joint name="j13" type="revolute">
@@ -464,5 +457,5 @@
         <origin xyz="0 0 0.04454" rpy="0 0 0" />
         <axis xyz="-1 0 0" />
-        <mimic joint="j9a_littlefinger" multiplier="1.35880" offset="0" />
+        <mimic joint="Pinky" multiplier="1.35880" offset="0" />
     </joint>
     <joint name="j17" type="revolute">
@@ -472,5 +465,12 @@
         <origin xyz="0 0 0.022" rpy="0 0 0" />
         <axis xyz="-1 0 0" />
-        <mimic joint="j9a_littlefinger" multiplier="1.42307" offset="0" />
+        <mimic joint="Pinky" multiplier="1.42307" offset="0" />
+    </joint>
+        <joint name="Finger_Spread" type="revolute">
+        <parent link="virtual_l" />
+        <child link="l" />
+        <limit effort="1000.0" lower="0.0" upper="0.28833" velocity="1" />
+        <origin xyz="0 0 0" rpy="0 0 0" />
+        <axis xyz="0 ${orientation*(-1)} 0" />
     </joint>
 </robot>

Commit message: fixed joints in urdf

File: s5fh_gripper/description/urdf/s5fs.urdf.xacro (robot description, xacro)
@@ -411,4 +411,52 @@
         <axis xyz="-1 0 0" />
     </joint>
+    <joint name="j12" type="revolute">
+        <parent link="j" />
+        <child link="n" />
+        <limit effort="1000.0" lower="0" upper="1.334" velocity="1" />
+        <origin xyz="0 0 0.05004" rpy="0 0 0" />
+        <axis xyz="-1 0 0" />
+        <mimic joint="Ring_Finger" multiplier="1.3588" offset="0" />
+    </joint>
+    <joint name="j16" type="revolute">
+        <parent link="n" />
+        <child link="r" />
+        <limit effort="1000.0" lower="0" upper="1.395" velocity="1" />
+        <origin xyz="0 0 0.032" rpy="0 0 0" />
+        <axis xyz="-1 0 0" />
+        <mimic joint="Ring_Finger" multiplier="1.42093" offset="0" />
+    </joint>
+    <!-- LITTLE FINGER JOINTS -->
+    <joint name="Pinky" type="revolute">
+        <parent link="e4" />
+        <child link="virtual_i" />
+        <limit effort="1000.0" lower="0.0" upper="0.98175" velocity="1" />
+        <origin xyz="0 0 0.056" rpy="0 0 0" />
+        <axis xyz="-1 0 0" />
+    </joint>
+    <joint name="j13" type="revolute">
+        <parent link="i" />
+        <child link="m" />
+        <limit effort="1000.0" lower="0" upper="1.334" velocity="1" />
+        <origin xyz="0 0 0.04454" rpy="0 0 0" />
+        <axis xyz="-1 0 0" />
+        <mimic joint="Pinky" multiplier="1.35880" offset="0" />
+    </joint>
+    <joint name="j17" type="revolute">
+        <parent link="m" />
+        <child link="q" />
+        <limit effort="1000.0" lower="0" upper="1.3971" velocity="1" />
+        <origin xyz="0 0 0.022" rpy="0 0 0" />
+        <axis xyz="-1 0 0" />
+        <mimic joint="Pinky" multiplier="1.42307" offset="0" />
+    </joint>
+        <joint name="j6b" type="revolute">
+        <parent link="virtual_l" />
+        <child link="l" />
+        <limit effort="1000.0" lower="0.0" upper="0.28833" velocity="1" />
+        <origin xyz="0 0 0" rpy="0 0 0" />
+        <axis xyz="0 ${orientation*(-1)} 0" />
+        <mimic joint="Finger_Spread" multiplier="0.5" offset="0" />
+    </joint>
     <joint name="j8b" type="revolute">
         <parent link="virtual_j" />
@@ -417,31 +465,7 @@
         <origin xyz="${orientation*(0.00675)} 0 0" rpy="0 0 0" />
         <axis xyz="0 ${orientation*(1)} 0" />
-        <mimic joint="Finger_Spread" multiplier="1" offset="0" />
-    </joint>
-    <joint name="j12" type="revolute">
-        <parent link="j" />
-        <child link="n" />
-        <limit effort="1000.0" lower="0" upper="1.334" velocity="1" />
-        <origin xyz="0 0 0.05004" rpy="0 0 0" />
-        <axis xyz="-1 0 0" />
-        <mimic joint="Ring_Finger" multiplier="1.3588" offset="0" />
-    </joint>
-    <joint name="j16" type="revolute">
-        <parent link="n" />
-        <child link="r" />
-        <limit effort="1000.0" lower="0" upper="1.395" velocity="1" />
-        <origin xyz="0 0 0.032" rpy="0 0 0" />
-        <axis xyz="-1 0 0" />
-        <mimic joint="Ring_Finger" multiplier="1.42093" offset="0" />
-    </joint>
-    <!-- LITTLE FINGER JOINTS -->
-    <joint name="Pinky" type="revolute">
-        <parent link="e4" />
-        <child link="virtual_i" />
-        <limit effort="1000.0" lower="0.0" upper="0.98175" velocity="1" />
-        <origin xyz="0 0 0.056" rpy="0 0 0" />
-        <axis xyz="-1 0 0" />
-    </joint>
-    <joint name="j9b" type="revolute">
+        <mimic joint="Finger_Spread" multiplier="0.5" offset="0" />
+    </joint>
+    <joint name="Finger_Spread" type="revolute">
         <parent link="virtual_i" />
         <child link="i" />
@@ -449,28 +473,4 @@
         <origin xyz="${orientation*(0.02825)} 0 0" rpy="0 0 0" />
         <axis xyz="0 ${orientation*(1)} 0" />
-        <mimic joint="Finger_Spread" multiplier="2.02164" offset="0" />
-    </joint>
-    <joint name="j13" type="revolute">
-        <parent link="i" />
-        <child link="m" />
-        <limit effort="1000.0" lower="0" upper="1.334" velocity="1" />
-        <origin xyz="0 0 0.04454" rpy="0 0 0" />
-        <axis xyz="-1 0 0" />
-        <mimic joint="Pinky" multiplier="1.35880" offset="0" />
-    </joint>
-    <joint name="j17" type="revolute">
-        <parent link="m" />
-        <child link="q" />
-        <limit effort="1000.0" lower="0" upper="1.3971" velocity="1" />
-        <origin xyz="0 0 0.022" rpy="0 0 0" />
-        <axis xyz="-1 0 0" />
-        <mimic joint="Pinky" multiplier="1.42307" offset="0" />
-    </joint>
-        <joint name="Finger_Spread" type="revolute">
-        <parent link="virtual_l" />
-        <child link="l" />
-        <limit effort="1000.0" lower="0.0" upper="0.28833" velocity="1" />
-        <origin xyz="0 0 0" rpy="0 0 0" />
-        <axis xyz="0 ${orientation*(-1)} 0" />
-    </joint>
+     </joint>
 </robot>

Commit message: attached hand to arm

File: s5fh_gripper/description/urdf/s5fs.urdf.xacro (robot description, xacro)
@@ -1,9 +1,15 @@
 <?xml version="1.0"?>
-<robot name="s5fs" xmlns:xacro="http://www.ros.org/wiki/xacro">
-    <xacro:property name="cyl_radius" value="0.001" />
-    <!-- RIGHT HAND = 1, LEFT HAND = -1 -->
-    <xacro:property name="orientation" value="-1" />
+<robot xmlns:xacro="http://www.ros.org/wiki/xacro">
+<xacro:property name="cyl_radius" value="0.001" />
+<xacro:macro name="s5fh" params="parent name side *origin">
+   <!-- RIGHT HAND = 1, LEFT HAND = -1 -->
     <!-- BASE_LINE LINKS -->
-    <link name="base_link">
+   <joint name="${name}_base_joint" type="fixed" >
+      <insert_block name="origin" />
+      <parent link="${parent}" />
+      <child link="${name}_base_link" />
+    </joint>
+    <link name="${name}_base_link">
+        <xacro:insert_block name="origin" />
         <visual>
             <origin rpy="0 0 0" xyz="0 0.01313 0" />
@@ -27,5 +33,5 @@
     <link name="h">
         <visual>
-            <origin rpy="0 1.571 0" xyz="${orientation*(-0.0125)} 0 0.0825" />
+            <origin rpy="0 1.571 0" xyz="${side*(-0.0125)} 0 0.0825" />
             <geometry>
                 <cylinder length="0.025" radius="${cyl_radius}" />
@@ -36,5 +42,5 @@
     <link name="d2">
         <visual>
-            <origin rpy="0 0 0" xyz="${orientation*(-0.025)} 0 0.09625" />
+            <origin rpy="0 0 0" xyz="${side*(-0.025)} 0 0.09625" />
             <geometry>
                 <cylinder length="0.0275" radius="${cyl_radius}" />
@@ -46,5 +52,5 @@
     <link name="e1">
         <visual>
-            <origin rpy="0 0 0" xyz="${orientation*(0.01840)} 0 0.01875" />
+            <origin rpy="0 0 0" xyz="${side*(0.01840)} 0 0.01875" />
             <geometry>
                 <cylinder length="0.0375" radius="${cyl_radius}" />
@@ -56,5 +62,5 @@
     <link name="e2">
         <visual>
-            <origin rpy="0 1.571 0" xyz="${orientation*(0.00875)} 0 0" />
+            <origin rpy="0 1.571 0" xyz="${side*(0.00875)} 0 0" />
             <geometry>
                 <cylinder length="0.0175" radius="${cyl_radius}" />
@@ -66,5 +72,5 @@
     <link name="e3">
         <visual>
-            <origin rpy="0 0 0" xyz="${orientation*(0.0175)} 0 0.015" />
+            <origin rpy="0 0 0" xyz="${side*(0.0175)} 0 0.015" />
             <geometry>
                 <cylinder length="0.03" radius="${cyl_radius}" />
@@ -75,5 +81,5 @@
     <link name="e">
         <visual>
-            <origin rpy="0 1.571 0" xyz="${orientation*(0.0175)} 0 0.03" />
+            <origin rpy="0 1.571 0" xyz="${side*(0.0175)} 0 0.03" />
             <geometry>
                 <cylinder length="0.0215" radius="${cyl_radius}" />
@@ -85,5 +91,5 @@
     <link name="e4">
         <visual>
-            <origin rpy="0 0 0" xyz="${orientation*(0.02825)} 0 0.043" />
+            <origin rpy="0 0 0" xyz="${side*(0.02825)} 0 0.043" />
             <geometry>
                 <cylinder length="0.026" radius="${cyl_radius}" />
@@ -95,5 +101,5 @@
     <link name="e5">
         <visual>
-            <origin rpy="0 0 0" xyz="${orientation*(0.00675)} 0 0.04775" />
+            <origin rpy="0 0 0" xyz="${side*(0.00675)} 0 0.04775" />
             <geometry>
                 <cylinder length="0.0355" radius="${cyl_radius}" />
@@ -280,17 +286,17 @@
         <limit effort="1000.0" lower="0.0" upper="0.9704" velocity="1" />
         <origin xyz="0 0 0.04596" rpy="0 0 0" />
-        <axis xyz="${orientation*(1)} 0 0" />
+        <axis xyz="${side*(1)} 0 0" />
     </joint>
     <!-- BASE_LINE JOINTS -->
     <joint name="Thumb_Opposition" type="revolute">
-        <parent link="base_link" />
+        <parent link="${name}_base_link" />
         <child link="z" />
         <limit effort="1000.0" lower="0.0" upper="0.9879" velocity="1" />
-        <origin xyz="${orientation*(-0.01690)} 0.02626 0" rpy="0 0.2618 1.571" />
-        <axis xyz="0 0 ${orientation*(-1)}" />
+        <origin xyz="${side*(-0.01690)} 0.02626 0" rpy="0 0.2618 1.571" />
+        <axis xyz="0 0 ${side*(-1)}" />
     </joint>
     <!-- JOINT NOT FOR BASE_LINE. BUT WRITTEN DOWN HERE FOR BETTER UX -->
     <joint name="f1" type="fixed">
-        <parent link="base_link" />
+        <parent link="${name}_base_link" />
         <child link="d" />
         <origin xyz="0 0 0" rpy="0 0 0" />
@@ -307,5 +313,5 @@
     </joint>
     <joint name="f4" type="fixed">
-        <parent link="base_link" />
+        <parent link="${name}_base_link" />
         <child link="e1" />
         <origin xyz="0 0 0" rpy="0 0 0" />
@@ -315,6 +321,6 @@
         <child link="e2" />
         <limit effort="1000.0" lower="0.0" upper="0.98786" velocity="1" />
-        <origin xyz="${orientation*(0.01840)} 0 0.0375" rpy="0 0 0" />
-        <axis xyz="0 0 ${orientation*(1)}" />
+        <origin xyz="${side*(0.01840)} 0 0.0375" rpy="0 0 0" />
+        <axis xyz="0 0 ${side*(1)}" />
         <mimic joint="Thumb_Opposition" multiplier="1" offset="0" />
     </joint>
@@ -345,5 +351,5 @@
         <limit effort="1000.0" lower="0.0" upper="0.98506" velocity="1" />
         <origin xyz="0 0 0.0485" rpy="0 0 0" />
-        <axis xyz="${orientation*(1)} 0 0" />
+        <axis xyz="${side*(1)} 0 0" />
         <mimic joint="Thumb_Flexion" multiplier="1.01511" offset="0" />
     </joint>
@@ -353,5 +359,5 @@
         <limit effort="1000.0" lower="0.0" upper="1.406" velocity="1" />
         <origin xyz="0 0 0.030" rpy="0 0 0" />
-        <axis xyz="${orientation*(1)} 0 0" />
+        <axis xyz="${side*(1)} 0 0" />
         <mimic joint="Thumb_Flexion" multiplier="1.44889" offset="0" />
     </joint>
@@ -368,5 +374,5 @@
         <child link="virtual_l" />
         <limit effort="1000.0" lower="0.0" upper="0.79849" velocity="1" />
-        <origin xyz="${orientation*(-0.025)} 0 0.110" rpy="0 0 0" />
+        <origin xyz="${side*(-0.025)} 0 0.110" rpy="0 0 0" />
         <axis xyz="-1 0 0" />
     </joint>
@@ -456,5 +462,5 @@
         <limit effort="1000.0" lower="0.0" upper="0.28833" velocity="1" />
         <origin xyz="0 0 0" rpy="0 0 0" />
-        <axis xyz="0 ${orientation*(-1)} 0" />
+        <axis xyz="0 ${side*(-1)} 0" />
         <mimic joint="Finger_Spread" multiplier="0.5" offset="0" />
     </joint>
@@ -463,6 +469,6 @@
         <child link="j" />
         <limit effort="1000.0" lower="0.0" upper="0.28833" velocity="1" />
-        <origin xyz="${orientation*(0.00675)} 0 0" rpy="0 0 0" />
-        <axis xyz="0 ${orientation*(1)} 0" />
+        <origin xyz="${side*(0.00675)} 0 0" rpy="0 0 0" />
+        <axis xyz="0 ${side*(1)} 0" />
         <mimic joint="Finger_Spread" multiplier="0.5" offset="0" />
     </joint>
@@ -471,6 +477,7 @@
         <child link="i" />
         <limit effort="1000.0" lower="0.0" upper="0.5829" velocity="1" />
-        <origin xyz="${orientation*(0.02825)} 0 0" rpy="0 0 0" />
-        <axis xyz="0 ${orientation*(1)} 0" />
+        <origin xyz="${side*(0.02825)} 0 0" rpy="0 0 0" />
+        <axis xyz="0 ${side*(1)} 0" />
      </joint>
+</xacro:macro>
 </robot>
