Commit message: fix orientation of thumb coordinate systems

File: s5fh_controller/description/urdf/s5fs.urdf.xacro (robot description, xacro)
@@ -15,6 +15,6 @@
             <origin rpy="0 0 0" xyz="0 0.01313 0" />
             <geometry>
-                <box size="0.0353 0.02626 0.010" />
-            </geometry>
+	      <mesh scale="0.001 0.001 0.001" filename="package://s5fh_controller/description/meshes/h10.dae" />
+	    </geometry>
             <material name="green">
                 <color rgba="0 1 0 1" />
@@ -285,6 +285,6 @@
         <child link="a" />
         <limit effort="1000.0" lower="0.0" upper="0.9704" velocity="1" />
-        <origin xyz="0 0 0.04596" rpy="0 0 0" />
-        <axis xyz="${side*(1)} 0 0" />
+        <origin xyz="0 0 0.04596" rpy="1.5707 0 1.5707" />
+        <axis xyz="0 0 ${side*(1)}" />
     </joint>
     <!-- BASE_LINE JOINTS -->
@@ -350,6 +350,6 @@
         <child link="b" />
         <limit effort="1000.0" lower="0.0" upper="0.98506" velocity="1" />
-        <origin xyz="0 0 0.0485" rpy="0 0 0" />
-        <axis xyz="${side*(1)} 0 0" />
+        <origin xyz="0 0.0485 0" rpy="0 0 0" />
+        <axis xyz="0 0 ${side*(1)}" />
         <mimic joint="Thumb_Flexion" multiplier="1.01511" offset="0" />
     </joint>
@@ -358,6 +358,6 @@
         <child link="c" />
         <limit effort="1000.0" lower="0.0" upper="1.406" velocity="1" />
-        <origin xyz="0 0 0.030" rpy="0 0 0" />
-        <axis xyz="${side*(1)} 0 0" />
+        <origin xyz="0 0.030 0" rpy="0 0 0" />
+        <axis xyz="0 0 ${side*(1)}" />
         <mimic joint="Thumb_Flexion" multiplier="1.44889" offset="0" />
     </joint>

Commit message: correct x axis for thumb and fix index finger

File: s5fh_controller/description/urdf/s5fs.urdf.xacro (robot description, xacro)
@@ -285,5 +285,5 @@
         <child link="a" />
         <limit effort="1000.0" lower="0.0" upper="0.9704" velocity="1" />
-        <origin xyz="0 0 0.04596" rpy="1.5707 0 1.5707" />
+        <origin xyz="0 0 0.04596" rpy="0 -1.5707 3.1415" />
         <axis xyz="0 0 ${side*(1)}" />
     </joint>
@@ -350,5 +350,5 @@
         <child link="b" />
         <limit effort="1000.0" lower="0.0" upper="0.98506" velocity="1" />
-        <origin xyz="0 0.0485 0" rpy="0 0 0" />
+        <origin xyz="0.0485 0 0" rpy="0 0 0" />
         <axis xyz="0 0 ${side*(1)}" />
         <mimic joint="Thumb_Flexion" multiplier="1.01511" offset="0" />
@@ -358,15 +358,15 @@
         <child link="c" />
         <limit effort="1000.0" lower="0.0" upper="1.406" velocity="1" />
-        <origin xyz="0 0.030 0" rpy="0 0 0" />
+        <origin xyz="0.030 0 0" rpy="0 0 0" />
         <axis xyz="0 0 ${side*(1)}" />
         <mimic joint="Thumb_Flexion" multiplier="1.44889" offset="0" />
     </joint>
-    <!-- FOREFINGER JOINTS -->
+    <!-- INDEX FINGER JOINTS -->
     <joint name="Index_Finger_Distal" type="revolute">
         <parent link="l" />
         <child link="p" />
         <limit effort="1000.0" lower="0" upper="1.334" velocity="1" />
-        <origin xyz="0 0 0.04804" rpy="0 0 0" />
-        <axis xyz="-1 0 0" />
+        <origin xyz="0.04804 0 0" rpy="1.5707 0 0" />
+        <axis xyz="0 0 1" />
     </joint>
     <joint name="Index_Finger_Proximal" type="revolute">
@@ -374,6 +374,6 @@
         <child link="virtual_l" />
         <limit effort="1000.0" lower="0.0" upper="0.79849" velocity="1" />
-        <origin xyz="${side*(-0.025)} 0 0.110" rpy="0 0 0" />
-        <axis xyz="-1 0 0" />
+        <origin xyz="${side*(-0.025)} 0 0.110" rpy="0 -1.5707 0" />
+        <axis xyz="0 0 1" />
     </joint>
     <!-- JOINT Finger_Spread in BASE_LINE section for better UX -->
@@ -382,6 +382,6 @@
         <child link="t" />
         <limit effort="1000.0" lower="0" upper="1.394" velocity="1" />
-        <origin xyz="0 0 0.026" rpy="0 0 0" />
-        <axis xyz="-1 0 0" />
+        <origin xyz="0.026 0 0" rpy="0 0 0" />
+        <axis xyz="0 0 1" />
         <mimic joint="Index_Finger_Distal" multiplier="1.0450" offset="0" />
     </joint>
@@ -461,6 +461,6 @@
         <child link="l" />
         <limit effort="1000.0" lower="0.0" upper="0.28833" velocity="1" />
-        <origin xyz="0 0 0" rpy="0 0 0" />
-        <axis xyz="0 ${side*(-1)} 0" />
+        <origin xyz="0 0 0" rpy="-1.5707 0 0" />
+        <axis xyz="0 0 ${side*(-1)}" />
         <mimic joint="Finger_Spread" multiplier="0.5" offset="0" />
     </joint>

Commit message: fix orientation of middle finger coordinate systems

File: s5fh_controller/description/urdf/s5fs.urdf.xacro (robot description, xacro)
@@ -387,17 +387,17 @@
     </joint>
     <!-- MIDDLE FINGER JOINTS -->
+    <joint name="Middle_Finger_Proximal" type="revolute">
+        <parent link="d" />
+        <child link="k" />
+        <limit effort="1000.0" lower="0.0" upper="0.79849" velocity="1" />
+        <origin xyz="0 0 0.110" rpy="0 -1.5707 0" />
+        <axis xyz="0 0 1" />
+    </joint>
     <joint name="Middle_Finger_Distal" type="revolute">
         <parent link="k" />
         <child link="o" />
         <limit effort="1000.0" lower="0" upper="1.334" velocity="1" />
-        <origin xyz="0 0 0.05004" rpy="0 0 0" />
-        <axis xyz="-1 0 0" />
-    </joint>
-    <joint name="Middle_Finger_Proximal" type="revolute">
-        <parent link="d" />
-        <child link="k" />
-        <limit effort="1000.0" lower="0.0" upper="0.79849" velocity="1" />
-        <origin xyz="0 0 0.110" rpy="0 0 0" />
-        <axis xyz="-1 0 0" />
+        <origin xyz="0.05004 0 0" rpy="0 0 0" />
+        <axis xyz="0 0 1" />
     </joint>
      <joint name="j15" type="revolute">
@@ -405,6 +405,6 @@
         <child link="s" />
         <limit effort="1000.0" lower="0" upper="1.334" velocity="1" />
-        <origin xyz="0 0 0.032" rpy="0 0 0" />
-        <axis xyz="-1 0 0" />
+        <origin xyz="0.032 0 0" rpy="0 0 0" />
+        <axis xyz="0 0 1" />
         <mimic joint="Middle_Finger_Distal" multiplier="1.000" offset="0" />
     </joint>

Commit message: fix orientation of ring finger coordinate systems

File: s5fh_controller/description/urdf/s5fs.urdf.xacro (robot description, xacro)
@@ -414,6 +414,6 @@
         <child link="virtual_j" />
         <limit effort="1000.0" lower="0.0" upper="0.98175" velocity="1" />
-        <origin xyz="0 0 0.0655" rpy="0 0 0" />
-        <axis xyz="-1 0 0" />
+        <origin xyz="0 0 0.0655" rpy="0 -1.5707 0" />
+        <axis xyz="0 0 1" />
     </joint>
     <joint name="j12" type="revolute">
@@ -421,6 +421,6 @@
         <child link="n" />
         <limit effort="1000.0" lower="0" upper="1.334" velocity="1" />
-        <origin xyz="0 0 0.05004" rpy="0 0 0" />
-        <axis xyz="-1 0 0" />
+        <origin xyz="0 -0.05004 0" rpy="1.5705 0 -1.5707" />
+        <axis xyz="0 0 1" />
         <mimic joint="Ring_Finger" multiplier="1.3588" offset="0" />
     </joint>
@@ -429,6 +429,6 @@
         <child link="r" />
         <limit effort="1000.0" lower="0" upper="1.395" velocity="1" />
-        <origin xyz="0 0 0.032" rpy="0 0 0" />
-        <axis xyz="-1 0 0" />
+        <origin xyz="0.032 0 0" rpy="0 0 0" />
+        <axis xyz="0 0 1" />
         <mimic joint="Ring_Finger" multiplier="1.42093" offset="0" />
     </joint>
@@ -469,6 +469,6 @@
         <child link="j" />
         <limit effort="1000.0" lower="0.0" upper="0.28833" velocity="1" />
-        <origin xyz="${side*(0.00675)} 0 0" rpy="0 0 0" />
-        <axis xyz="0 ${side*(1)} 0" />
+        <origin xyz="0 0 ${side*(-0.00675)}" rpy="${side*(-1.5707)} ${side*(1.5707)} 0" />
+        <axis xyz="0 0 1" />
         <mimic joint="Finger_Spread" multiplier="0.5" offset="0" />
     </joint>

Commit message: fix orientation of pinky coordinate systems

File: s5fh_controller/description/urdf/s5fs.urdf.xacro (robot description, xacro)
@@ -438,6 +438,6 @@
         <child link="virtual_i" />
         <limit effort="1000.0" lower="0.0" upper="0.98175" velocity="1" />
-        <origin xyz="0 0 0.056" rpy="0 0 0" />
-        <axis xyz="-1 0 0" />
+        <origin xyz="0 0 0.056" rpy="0 -1.5707 0" />
+        <axis xyz="0 0 1" />
     </joint>
     <joint name="j13" type="revolute">
@@ -445,6 +445,6 @@
         <child link="m" />
         <limit effort="1000.0" lower="0" upper="1.334" velocity="1" />
-        <origin xyz="0 0 0.04454" rpy="0 0 0" />
-        <axis xyz="-1 0 0" />
+        <origin xyz="0 -0.04454 0" rpy="1.5705 0 -1.5707" />
+        <axis xyz="0 0 1" />
         <mimic joint="Pinky" multiplier="1.35880" offset="0" />
     </joint>
@@ -453,6 +453,6 @@
         <child link="q" />
         <limit effort="1000.0" lower="0" upper="1.3971" velocity="1" />
-        <origin xyz="0 0 0.022" rpy="0 0 0" />
-        <axis xyz="-1 0 0" />
+        <origin xyz="0.022 0 0" rpy="0 0 0" />
+        <axis xyz="0 0 1" />
         <mimic joint="Pinky" multiplier="1.42307" offset="0" />
     </joint>
@@ -477,6 +477,6 @@
         <child link="i" />
         <limit effort="1000.0" lower="0.0" upper="0.5829" velocity="1" />
-        <origin xyz="${side*(0.02825)} 0 0" rpy="0 0 0" />
-        <axis xyz="0 ${side*(1)} 0" />
+        <origin xyz="0 0 ${side*(-0.02825)}" rpy="${side*(-1.5707)} ${side *(1.5707)} 0" />
+        <axis xyz="0 0 1" />
      </joint>
 </xacro:macro>

Commit message: fix left hand (i.e. size == -1) ring finger and pinky movement

File: s5fh_controller/description/urdf/s5fs.urdf.xacro (robot description, xacro)
@@ -469,6 +469,6 @@
         <child link="j" />
         <limit effort="1000.0" lower="0.0" upper="0.28833" velocity="1" />
-        <origin xyz="0 0 ${side*(-0.00675)}" rpy="${side*(-1.5707)} ${side*(1.5707)} 0" />
-        <axis xyz="0 0 1" />
+        <origin xyz="0 0 ${side*(-0.00675)}" rpy="-1.5707 1.5707 0" />
+        <axis xyz="0 0 ${side*(1)}" />
         <mimic joint="Finger_Spread" multiplier="0.5" offset="0" />
     </joint>
@@ -477,6 +477,6 @@
         <child link="i" />
         <limit effort="1000.0" lower="0.0" upper="0.5829" velocity="1" />
-        <origin xyz="0 0 ${side*(-0.02825)}" rpy="${side*(-1.5707)} ${side *(1.5707)} 0" />
-        <axis xyz="0 0 1" />
+        <origin xyz="0 0 ${side*(-0.02825)}" rpy="-1.5707 1.5707 0" />
+        <axis xyz="0 0 ${side*(1)}" />
      </joint>
 </xacro:macro>
