Commit message: switch spread and tilt joins for pinky, index and ring finger, add models, unify indentation
models aren't currently oriented correctly and have some wrong normals - this will be changed soon

File: s5fh_controller/description/urdf/s5fs.urdf.xacro (robot description, xacro)
@@ -1,9 +1,9 @@
 <?xml version="1.0"?>
 <robot xmlns:xacro="http://www.ros.org/wiki/xacro">
-<xacro:property name="cyl_radius" value="0.001" />
-<xacro:macro name="s5fh" params="parent name side *origin">
-   <!-- RIGHT HAND = 1, LEFT HAND = -1 -->
+  <xacro:property name="cyl_radius" value="0.001" />
+  <xacro:macro name="s5fh" params="parent name side *origin">
+    <!-- RIGHT HAND = 1, LEFT HAND = -1 -->
     <!-- BASE_LINE LINKS -->
-   <joint name="${name}_base_joint" type="fixed" >
+    <joint name="${name}_base_joint" type="fixed" >
       <insert_block name="origin" />
       <parent link="${parent}" />
@@ -11,473 +11,474 @@
     </joint>
     <link name="${name}_base_link">
-        <xacro:insert_block name="origin" />
-        <visual>
-            <origin rpy="0 0 0" xyz="0 0.01313 0" />
-            <geometry>
-	      <mesh scale="0.001 0.001 0.001" filename="package://s5fh_controller/description/meshes/h10.dae" />
-	    </geometry>
-            <material name="green">
-                <color rgba="0 1 0 1" />
-            </material>
-        </visual>
+      <xacro:insert_block name="origin" />
+      <visual>
+	<origin rpy="0 0 0" xyz="0 0.01313 0" />
+	<geometry>
+	  <mesh scale="0.001 0.001 0.001" filename="package://s5fh_controller/description/meshes/h10.dae" />
+	</geometry>
+	<material name="green">
+	  <color rgba="0 1 0 1" />
+	</material>
+      </visual>
     </link>
     <link name="d">
-        <visual>
-            <origin rpy="0 0 0" xyz="0 0 0.055" />
-            <geometry>
-                <cylinder length="0.110" radius="${cyl_radius}" />
-            </geometry>
-            <material name="green" />
-        </visual>
+      <visual>
+	<origin rpy="0 0 0" xyz="0 0 0.055" />
+	<geometry>
+	  <cylinder length="0.110" radius="${cyl_radius}" />
+	</geometry>
+	<material name="green" />
+      </visual>
     </link>
     <link name="h">
-        <visual>
-            <origin rpy="0 1.571 0" xyz="${side*(-0.0125)} 0 0.0825" />
-            <geometry>
-                <cylinder length="0.025" radius="${cyl_radius}" />
-            </geometry>
-            <material name="green" />
-        </visual>
+      <visual>
+	<origin rpy="0 1.571 0" xyz="${side*(-0.0125)} 0 0.0825" />
+	<geometry>
+	  <cylinder length="0.025" radius="${cyl_radius}" />
+	</geometry>
+	<material name="green" />
+      </visual>
     </link>
     <link name="d2">
-        <visual>
-            <origin rpy="0 0 0" xyz="${side*(-0.025)} 0 0.09625" />
-            <geometry>
-                <cylinder length="0.0275" radius="${cyl_radius}" />
-            </geometry>
-            <material name="green" />
-        </visual>
+      <visual>
+	<origin rpy="0 0 0" xyz="${side*(-0.025)} 0 0.09625" />
+	<geometry>
+	  <cylinder length="0.0275" radius="${cyl_radius}" />
+	</geometry>
+	<material name="green" />
+      </visual>
     </link>
     <!-- LENGTH NOT FOUND IN DATASHEET! GUESSED!!! -->
     <link name="e1">
-        <visual>
-            <origin rpy="0 0 0" xyz="${side*(0.01840)} 0 0.01875" />
-            <geometry>
-                <cylinder length="0.0375" radius="${cyl_radius}" />
-            </geometry>
-            <material name="green" />
-        </visual>
+      <visual>
+	<origin rpy="0 0 0" xyz="${side*(0.01840)} 0 0.01875" />
+	<geometry>
+	  <cylinder length="0.0375" radius="${cyl_radius}" />
+	</geometry>
+	<material name="green" />
+      </visual>
     </link>
     <!-- LENGTH NOT FOUND IN DATASHEET! GUESSED!!! -->
     <link name="e2">
-        <visual>
-            <origin rpy="0 1.571 0" xyz="${side*(0.00875)} 0 0" />
-            <geometry>
-                <cylinder length="0.0175" radius="${cyl_radius}" />
-            </geometry>
-            <material name="green" />
-        </visual>
+      <visual>
+	<origin rpy="0 1.571 0" xyz="${side*(0.00875)} 0 0" />
+	<geometry>
+	  <cylinder length="0.0175" radius="${cyl_radius}" />
+	</geometry>
+	<material name="green" />
+      </visual>
     </link>
     <!-- LENGTH NOT FOUND IN DATASHEET! GUESSED!!! -->
     <link name="e3">
-        <visual>
-            <origin rpy="0 0 0" xyz="${side*(0.0175)} 0 0.015" />
-            <geometry>
-                <cylinder length="0.03" radius="${cyl_radius}" />
-            </geometry>
-            <material name="green" />
-        </visual>
+      <visual>
+	<origin rpy="0 0 0" xyz="${side*(0.0175)} 0 0.015" />
+	<geometry>
+	  <cylinder length="0.03" radius="${cyl_radius}" />
+	</geometry>
+	<material name="green" />
+      </visual>
     </link>
     <link name="e">
-        <visual>
-            <origin rpy="0 1.571 0" xyz="${side*(0.0175)} 0 0.03" />
-            <geometry>
-                <cylinder length="0.0215" radius="${cyl_radius}" />
-            </geometry>
-            <material name="green" />
-        </visual>
+      <visual>
+	<origin rpy="0 1.571 0" xyz="${side*(0.0175)} 0 0.03" />
+	<geometry>
+	  <cylinder length="0.0215" radius="${cyl_radius}" />
+	</geometry>
+	<material name="green" />
+      </visual>
     </link>
     <!-- LENGTH NOT FOUND IN DATASHEET! GUESSED, BUT POSITION CALCULATED: E4 = D-G-F!!! -->
     <link name="e4">
-        <visual>
-            <origin rpy="0 0 0" xyz="${side*(0.02825)} 0 0.043" />
-            <geometry>
-                <cylinder length="0.026" radius="${cyl_radius}" />
-            </geometry>
-            <material name="green" />
-        </visual>
+      <visual>
+	<origin rpy="0 0 0" xyz="${side*(0.02825)} 0 0.043" />
+	<geometry>
+	  <cylinder length="0.026" radius="${cyl_radius}" />
+	</geometry>
+	<material name="green" />
+      </visual>
     </link>
     <!-- LENGTH NOT FOUND IN DATASHEET! GUESSED, BUT POSITION CALCULATED: E5 = D-G!!! -->
     <link name="e5">
-        <visual>
-            <origin rpy="0 0 0" xyz="${side*(0.00675)} 0 0.04775" />
-            <geometry>
-                <cylinder length="0.0355" radius="${cyl_radius}" />
-            </geometry>
-            <material name="green" />
-        </visual>
+      <visual>
+	<origin rpy="0 0 0" xyz="${side*(0.00675)} 0 0.04775" />
+	<geometry>
+	  <cylinder length="0.0355" radius="${cyl_radius}" />
+	</geometry>
+	<material name="green" />
+      </visual>
     </link>
     <!-- THUMB LINKS -->
     <link name="z">
-        <visual>
-            <origin rpy="0 0 0" xyz="0 0 0.02298" />
-            <geometry>
-                <cylinder length="0.04596" radius="${cyl_radius}" />
-            </geometry>
-            <material name="green" />
-        </visual>
+      <visual>
+	<origin rpy="0 0 0" xyz="0 0 0.02298" />
+	<geometry>
+	  <mesh scale="0.001 0.001 0.001" filename="package://s5fh_controller/description/meshes/d10.dae" />
+	</geometry>
+	<material name="green" />
+      </visual>
     </link>
     <link name="a">
-        <visual>
-            <origin rpy="0 0 0" xyz="0 0 0.02425" />
-            <geometry>
-                <cylinder length="0.0485" radius="${cyl_radius}" />
-            </geometry>
-            <material name="green" />
-        </visual>
+      <visual>
+	<origin rpy="0 0 0" xyz="0 0 0.02425" />
+	<geometry>
+	  <mesh scale="0.001 0.001 0.001" filename="package://s5fh_controller/description/meshes/d11.dae" />
+	</geometry>
+	<material name="green" />
+      </visual>
     </link>
     <link name="b">
-        <visual>
-            <origin rpy="0 0 0" xyz="0 0 0.015" />
-            <geometry>
-                <cylinder length="0.030" radius="${cyl_radius}" />
-            </geometry>
-            <material name="green" />
-        </visual>
+      <visual>
+	<origin rpy="0 0 0" xyz="0 0 0.015" />
+	<geometry>
+	  <mesh scale="0.001 0.001 0.001" filename="package://s5fh_controller/description/meshes/d12.dae" />
+	</geometry>
+	<material name="green" />
+      </visual>
     </link>
     <link name="c">
-        <visual>
-            <origin rpy="0 0 0" xyz="0 0 0.010" />
-            <geometry>
-                <cylinder length="0.020" radius="${cyl_radius}" />
-            </geometry>
-            <material name="green" />
-        </visual>
-    </link>
-    <!-- FOREFINGER LINKS -->
+      <visual>
+	<origin rpy="0 0 0" xyz="0 0 0.010" />
+	<geometry>
+	  <mesh scale="0.001 0.001 0.001" filename="package://s5fh_controller/description/meshes/d13.dae" />
+	</geometry>
+	<material name="green" />
+      </visual>
+    </link>
+    <!-- INDEX FINGER LINKS -->
     <link name="virtual_l">
-        <visual>
-            <origin rpy="0 0 0" xyz="0 0 0" />
-            <geometry>
-                <cylinder length="0" radius="0" />
-            </geometry>
-        </visual>
+      <visual>
+	<origin rpy="0 0 0" xyz="0 0 0" />
+	<geometry>
+	  <mesh scale="0.001 0.001 0.001" filename="package://s5fh_controller/description/meshes/f10.dae" />
+	</geometry>
+      </visual>
     </link>
     <link name="l">
-        <visual>
-            <origin rpy="0 0 0" xyz="0 0 0.02402" />
-            <geometry>
-                <cylinder length="0.04804" radius="${cyl_radius}" />
-            </geometry>
-            <material name="green" />
-        </visual>
+      <visual>
+	<origin rpy="0 0 0" xyz="0 0 0.02402" />
+	<geometry>
+	  <mesh scale="0.001 0.001 0.001" filename="package://s5fh_controller/description/meshes/f11.dae" />
+	</geometry>
+	<material name="green" />
+      </visual>
     </link>
     <link name="p">
-        <visual>
-            <origin rpy="0 0 0" xyz="0 0 0.013" />
-            <geometry>
-                <cylinder length="0.026" radius="${cyl_radius}" />
-            </geometry>
-            <material name="green" />
-        </visual>
+      <visual>
+	<origin rpy="0 0 0" xyz="0 0 0.013" />
+	<geometry>
+	  <mesh scale="0.001 0.001 0.001" filename="package://s5fh_controller/description/meshes/f12.dae" />
+	</geometry>
+	<material name="green" />
+      </visual>
     </link>
     <link name="t">
-        <visual>
-            <origin rpy="0 0 0" xyz="0 0 0.0075" />
-            <geometry>
-                <cylinder length="0.015" radius="${cyl_radius}" />
-            </geometry>
-            <material name="green" />
-        </visual>
+      <visual>
+	<origin rpy="0 0 0" xyz="0 0 0.0075" />
+	<geometry>
+	  <mesh scale="0.001 0.001 0.001" filename="package://s5fh_controller/description/meshes/f13.dae" />
+	</geometry>
+	<material name="green" />
+      </visual>
     </link>
     <!-- MIDDLE FINGER LINKS -->
+    <!-- TODO(nberg): Add link for finger mount point (f20.dae) -->
     <link name="k">
-        <visual>
-            <origin rpy="0 0 0" xyz="0 0 0.02502" />
-            <geometry>
-                <cylinder length="0.05004" radius="${cyl_radius}" />
-            </geometry>
-            <material name="green" />
-        </visual>
+      <visual>
+	<origin rpy="0 0 0" xyz="0 0 0.02502" />
+	<geometry>
+	  <mesh scale="0.001 0.001 0.001" filename="package://s5fh_controller/description/meshes/f21.dae" />
+	</geometry>
+	<material name="green" />
+      </visual>
     </link>
     <link name="o">
-        <visual>
-            <origin rpy="0 0 0" xyz="0 0 0.016" />
-            <geometry>
-                <cylinder length="0.032" radius="${cyl_radius}" />
-            </geometry>
-            <material name="green" />
-        </visual>
+      <visual>
+	<origin rpy="0 0 0" xyz="0 0 0.016" />
+	<geometry>
+	  <mesh scale="0.001 0.001 0.001" filename="package://s5fh_controller/description/meshes/f22.dae" />
+	</geometry>
+	<material name="green" />
+      </visual>
     </link>
     <link name="s">
-        <visual>
-            <origin rpy="0 0 0" xyz="0 0 0.0075" />
-            <geometry>
-                <cylinder length="0.015" radius="${cyl_radius}" />
-            </geometry>
-            <material name="green" />
-        </visual>
+      <visual>
+	<origin rpy="0 0 0" xyz="0 0 0.0075" />
+	<geometry>
+	  <mesh scale="0.001 0.001 0.001" filename="package://s5fh_controller/description/meshes/f23.dae" />
+	</geometry>
+	<material name="green" />
+      </visual>
     </link>
     <!-- RING FINGER LINKS -->
     <link name="virtual_j">
-        <visual>
-            <origin rpy="0 0 0" xyz="0.006625 0 0" />
-            <geometry>
-                <cylinder length="0" radius="0" />
-            </geometry>
-        </visual>
+      <visual>
+	<origin rpy="0 0 0" xyz="0.006625 0 0" />
+	<geometry>
+	  <mesh scale="0.001 0.001 0.001" filename="package://s5fh_controller/description/meshes/f30.dae" />
+	</geometry>
+      </visual>
     </link>
     <link name="j">
-        <visual>
-            <origin rpy="0 0 0" xyz="0 0 0.02502" />
-            <geometry>
-                <cylinder length="0.05004" radius="${cyl_radius}" />
-            </geometry>
-            <material name="green" />
-        </visual>
+      <visual>
+	<origin rpy="0 0 0" xyz="0 0 0.02502" />
+	<geometry>
+	  <mesh scale="0.001 0.001 0.001" filename="package://s5fh_controller/description/meshes/f31.dae" />
+	</geometry>
+	<material name="green" />
+      </visual>
     </link>
     <link name="n">
-        <visual>
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
Commit message: add virtual middle finger "spread" link

File: s5fh_controller/description/urdf/s5fs.urdf.xacro (robot description, xacro)
@@ -182,5 +182,11 @@
     </link>
     <!-- MIDDLE FINGER LINKS -->
-    <!-- TODO(nberg): Add link for finger mount point (f20.dae) -->
+    <link name="virtual_k">
+      <visual>
+	<geometry>
+	  <mesh scale="0.001 0.001 0.001" filename="package://s5fh_controller/description/meshes/f20.dae" />
+	</geometry>
+      </visual>
+    </link>
     <link name="k">
       <visual>
@@ -389,8 +395,8 @@
     <!-- MIDDLE FINGER JOINTS -->
     <joint name="Middle_Finger_Proximal" type="revolute">
-      <parent link="d" />
+      <parent link="virtual_k" />
       <child link="k" />
       <limit effort="1000.0" lower="0.0" upper="0.79849" velocity="1" />
-      <origin xyz="0 0 0.110" rpy="0 -1.5707 0" />
+      <origin xyz="0 0 0" rpy="-1.5707 0 0" />
       <axis xyz="0 0 1" />
     </joint>
@@ -466,4 +472,9 @@
       <mimic joint="Finger_Spread" multiplier="0.5" offset="0" />
     </joint>
+    <joint name="middle_spread_dummy" type="fixed">
+      <parent link="d" />
+      <child link="virtual_k" />
+      <origin xyz="0 0 0.110" rpy="0 -1.5707 1.5707" />
+    </joint>
     <joint name="ring_spread" type="revolute">
       <parent link="e5" />

Commit message: Deleted wrongly rotated STLs and added new versions of the DAEs. Dropped scaling factor.

File: s5fh_controller/description/urdf/s5fs.urdf.xacro (robot description, xacro)
@@ -15,5 +15,5 @@
 	<origin rpy="0 0 0" xyz="0 0.01313 0" />
 	<geometry>
-	  <mesh scale="0.001 0.001 0.001" filename="package://s5fh_controller/description/meshes/h10.dae" />
+	  <mesh filename="package://s5fh_controller/description/meshes/h10.dae" />
 	</geometry>
 	<material name="green">
@@ -113,5 +113,5 @@
 	<origin rpy="0 0 0" xyz="0 0 0.02298" />
 	<geometry>
-	  <mesh scale="0.001 0.001 0.001" filename="package://s5fh_controller/description/meshes/d10.dae" />
+	  <mesh filename="package://s5fh_controller/description/meshes/d10.dae" />
 	</geometry>
 	<material name="green" />
@@ -122,5 +122,5 @@
 	<origin rpy="0 0 0" xyz="0 0 0.02425" />
 	<geometry>
-	  <mesh scale="0.001 0.001 0.001" filename="package://s5fh_controller/description/meshes/d11.dae" />
+	  <mesh filename="package://s5fh_controller/description/meshes/d11.dae" />
 	</geometry>
 	<material name="green" />
@@ -131,5 +131,5 @@
 	<origin rpy="0 0 0" xyz="0 0 0.015" />
 	<geometry>
-	  <mesh scale="0.001 0.001 0.001" filename="package://s5fh_controller/description/meshes/d12.dae" />
+	  <mesh filename="package://s5fh_controller/description/meshes/d12.dae" />
 	</geometry>
 	<material name="green" />
@@ -140,5 +140,5 @@
 	<origin rpy="0 0 0" xyz="0 0 0.010" />
 	<geometry>
-	  <mesh scale="0.001 0.001 0.001" filename="package://s5fh_controller/description/meshes/d13.dae" />
+	  <mesh filename="package://s5fh_controller/description/meshes/d13.dae" />
 	</geometry>
 	<material name="green" />
@@ -150,5 +150,5 @@
 	<origin rpy="0 0 0" xyz="0 0 0" />
 	<geometry>
-	  <mesh scale="0.001 0.001 0.001" filename="package://s5fh_controller/description/meshes/f10.dae" />
+	  <mesh filename="package://s5fh_controller/description/meshes/f10.dae" />
 	</geometry>
       </visual>
@@ -158,5 +158,5 @@
 	<origin rpy="0 0 0" xyz="0 0 0.02402" />
 	<geometry>
-	  <mesh scale="0.001 0.001 0.001" filename="package://s5fh_controller/description/meshes/f11.dae" />
+	  <mesh filename="package://s5fh_controller/description/meshes/f11.dae" />
 	</geometry>
 	<material name="green" />
@@ -167,5 +167,5 @@
 	<origin rpy="0 0 0" xyz="0 0 0.013" />
 	<geometry>
-	  <mesh scale="0.001 0.001 0.001" filename="package://s5fh_controller/description/meshes/f12.dae" />
+	  <mesh filename="package://s5fh_controller/description/meshes/f12.dae" />
 	</geometry>
 	<material name="green" />
@@ -176,5 +176,5 @@
 	<origin rpy="0 0 0" xyz="0 0 0.0075" />
 	<geometry>
-	  <mesh scale="0.001 0.001 0.001" filename="package://s5fh_controller/description/meshes/f13.dae" />
+	  <mesh filename="package://s5fh_controller/description/meshes/f13.dae" />
 	</geometry>
 	<material name="green" />
@@ -185,5 +185,5 @@
       <visual>
 	<geometry>
-	  <mesh scale="0.001 0.001 0.001" filename="package://s5fh_controller/description/meshes/f20.dae" />
+	  <mesh filename="package://s5fh_controller/description/meshes/f20.dae" />
 	</geometry>
       </visual>
@@ -193,5 +193,5 @@
 	<origin rpy="0 0 0" xyz="0 0 0.02502" />
 	<geometry>
-	  <mesh scale="0.001 0.001 0.001" filename="package://s5fh_controller/description/meshes/f21.dae" />
+	  <mesh filename="package://s5fh_controller/description/meshes/f21.dae" />
 	</geometry>
 	<material name="green" />
@@ -202,5 +202,5 @@
 	<origin rpy="0 0 0" xyz="0 0 0.016" />
 	<geometry>
-	  <mesh scale="0.001 0.001 0.001" filename="package://s5fh_controller/description/meshes/f22.dae" />
+	  <mesh filename="package://s5fh_controller/description/meshes/f22.dae" />
 	</geometry>
 	<material name="green" />
@@ -211,5 +211,5 @@
 	<origin rpy="0 0 0" xyz="0 0 0.0075" />
 	<geometry>
-	  <mesh scale="0.001 0.001 0.001" filename="package://s5fh_controller/description/meshes/f23.dae" />
+	  <mesh filename="package://s5fh_controller/description/meshes/f23.dae" />
 	</geometry>
 	<material name="green" />
@@ -221,5 +221,5 @@
 	<origin rpy="0 0 0" xyz="0.006625 0 0" />
 	<geometry>
-	  <mesh scale="0.001 0.001 0.001" filename="package://s5fh_controller/description/meshes/f30.dae" />
+	  <mesh filename="package://s5fh_controller/description/meshes/f30.dae" />
 	</geometry>
       </visual>
@@ -229,5 +229,5 @@
 	<origin rpy="0 0 0" xyz="0 0 0.02502" />
 	<geometry>
-	  <mesh scale="0.001 0.001 0.001" filename="package://s5fh_controller/description/meshes/f31.dae" />
+	  <mesh filename="package://s5fh_controller/description/meshes/f31.dae" />
 	</geometry>
 	<material name="green" />
@@ -238,5 +238,5 @@
 	<origin rpy="0 0 0" xyz="0 0 0.01525" />
 	<geometry>
-	  <mesh scale="0.001 0.001 0.001" filename="package://s5fh_controller/description/meshes/f32.dae" />
+	  <mesh filename="package://s5fh_controller/description/meshes/f32.dae" />
 	</geometry>
 	<material name="green" />
@@ -247,5 +247,5 @@
 	<origin rpy="0 0 0" xyz="0 0 0.00675" />
 	<geometry>
-	  <mesh scale="0.001 0.001 0.001" filename="package://s5fh_controller/description/meshes/f33.dae" />
+	  <mesh filename="package://s5fh_controller/description/meshes/f33.dae" />
 	</geometry>
 	<material name="green" />
@@ -257,5 +257,5 @@
 	<origin rpy="0 0 0" xyz="0.02825 0 0" />
 	<geometry>
-	  <mesh scale="0.001 0.001 0.001" filename="package://s5fh_controller/description/meshes/f40.dae" />
+	  <mesh filename="package://s5fh_controller/description/meshes/f40.dae" />
 	</geometry>
       </visual>
@@ -265,5 +265,5 @@
 	<origin rpy="0 0 0" xyz="0 0 0.02227" />
 	<geometry>
-	  <mesh scale="0.001 0.001 0.001" filename="package://s5fh_controller/description/meshes/f41.dae" />
+	  <mesh filename="package://s5fh_controller/description/meshes/f41.dae" />
 	</geometry>
 	<material name="green" />
@@ -274,5 +274,5 @@
 	<origin rpy="0 0 0" xyz="0 0 0.011" />
 	<geometry>
-	  <mesh scale="0.001 0.001 0.001" filename="package://s5fh_controller/description/meshes/f42.dae" />
+	  <mesh filename="package://s5fh_controller/description/meshes/f42.dae" />
 	</geometry>
 	<material name="green" />
@@ -283,5 +283,5 @@
 	<origin rpy="0 0 0" xyz="0 0 0.0075" />
 	<geometry>
-	  <mesh scale="0.001 0.001 0.001" filename="package://s5fh_controller/description/meshes/f43.dae" />
+	  <mesh filename="package://s5fh_controller/description/meshes/f43.dae" />
 	</geometry>
 	<material name="green" />
