Commit message: URDF fine tuning

File: s5fh_controller/description/urdf/s5fs.urdf.xacro (robot description, xacro)
@@ -13,7 +13,7 @@
       <xacro:insert_block name="origin" />
       <visual>
-	<origin rpy="0 0 0" xyz="0 0.01313 0" />
-	<geometry>
-	  <mesh filename="package://s5fh_controller/description/meshes/h10.dae" />
+	<origin xyz="0 0 -0.032" rpy="0 0 0" />
+	<geometry>
+	  <mesh filename="package://s5fh_controller/description/meshes/base10.dae" />
 	</geometry>
 	<material name="green">
@@ -24,5 +24,4 @@
     <link name="d">
       <visual>
-	<origin rpy="0 0 0" xyz="0 0 0.055" />
 	<geometry>
 	  <cylinder length="0.110" radius="${cyl_radius}" />
@@ -52,9 +51,8 @@
     <link name="e1">
       <visual>
-	<origin rpy="0 0 0" xyz="${side*(0.01840)} 0 0.01875" />
-	<geometry>
-	  <cylinder length="0.0375" radius="${cyl_radius}" />
-	</geometry>
-	<material name="green" />
+	<origin rpy="0 0 0" xyz="0 0.01313 0" />
+	<geometry>
+	  <mesh filename="package://s5fh_controller/description/meshes/h10.dae" />
+	</geometry>
       </visual>
     </link>
@@ -62,9 +60,8 @@
     <link name="e2">
       <visual>
-	<origin rpy="0 1.571 0" xyz="${side*(0.00875)} 0 0" />
-	<geometry>
-	  <cylinder length="0.0175" radius="${cyl_radius}" />
-	</geometry>
-	<material name="green" />
+	<origin xyz="-0.0007 0 -0.01002" />
+	<geometry>
+	  <mesh filename="package://s5fh_controller/description/meshes/h11.dae" />
+	</geometry>
       </visual>
     </link>
@@ -80,11 +77,4 @@
     </link>
     <link name="e">
-      <visual>
-	<origin rpy="0 1.571 0" xyz="${side*(0.0175)} 0 0.03" />
-	<geometry>
-	  <cylinder length="0.0215" radius="${cyl_radius}" />
-	</geometry>
-	<material name="green" />
-      </visual>
     </link>
     <!-- LENGTH NOT FOUND IN DATASHEET! GUESSED, BUT POSITION CALCULATED: E4 = D-G-F!!! -->
@@ -111,5 +101,5 @@
     <link name="z">
       <visual>
-	<origin rpy="0 0 0" xyz="0 0 0.02298" />
+	<origin xyz="0 0 0.02442" />
 	<geometry>
 	  <mesh filename="package://s5fh_controller/description/meshes/d10.dae" />
@@ -118,7 +108,7 @@
       </visual>
     </link>
+    <link name="virtual_a" />
     <link name="a">
       <visual>
-	<origin rpy="0 0 0" xyz="0 0 0.02425" />
 	<geometry>
 	  <mesh filename="package://s5fh_controller/description/meshes/d11.dae" />
@@ -129,5 +119,4 @@
     <link name="b">
       <visual>
-	<origin rpy="0 0 0" xyz="0 0 0.015" />
 	<geometry>
 	  <mesh filename="package://s5fh_controller/description/meshes/d12.dae" />
@@ -138,5 +127,4 @@
     <link name="c">
       <visual>
-	<origin rpy="0 0 0" xyz="0 0 0.010" />
 	<geometry>
 	  <mesh filename="package://s5fh_controller/description/meshes/d13.dae" />
@@ -148,5 +136,5 @@
     <link name="virtual_l">
       <visual>
-	<origin rpy="0 0 0" xyz="0 0 0" />
+	<origin xyz="0 0 0.01321" />
 	<geometry>
 	  <mesh filename="package://s5fh_controller/description/meshes/f10.dae" />
@@ -156,5 +144,4 @@
     <link name="l">
       <visual>
-	<origin rpy="0 0 0" xyz="0 0 0.02402" />
 	<geometry>
 	  <mesh filename="package://s5fh_controller/description/meshes/f11.dae" />
@@ -165,5 +152,4 @@
     <link name="p">
       <visual>
-	<origin rpy="0 0 0" xyz="0 0 0.013" />
 	<geometry>
 	  <mesh filename="package://s5fh_controller/description/meshes/f12.dae" />
@@ -174,5 +160,4 @@
     <link name="t">
       <visual>
-	<origin rpy="0 0 0" xyz="0 0 0.0075" />
 	<geometry>
 	  <mesh filename="package://s5fh_controller/description/meshes/f13.dae" />
@@ -184,4 +169,5 @@
     <link name="virtual_k">
       <visual>
+	<origin xyz="0 0 0.01321" />
 	<geometry>
 	  <mesh filename="package://s5fh_controller/description/meshes/f20.dae" />
@@ -191,5 +177,4 @@
     <link name="k">
       <visual>
-	<origin rpy="0 0 0" xyz="0 0 0.02502" />
 	<geometry>
 	  <mesh filename="package://s5fh_controller/description/meshes/f21.dae" />
@@ -200,5 +185,4 @@
     <link name="o">
       <visual>
-	<origin rpy="0 0 0" xyz="0 0 0.016" />
 	<geometry>
 	  <mesh filename="package://s5fh_controller/description/meshes/f22.dae" />
@@ -209,5 +193,4 @@
     <link name="s">
       <visual>
-	<origin rpy="0 0 0" xyz="0 0 0.0075" />
 	<geometry>
 	  <mesh filename="package://s5fh_controller/description/meshes/f23.dae" />
@@ -219,5 +202,5 @@
     <link name="virtual_j">
       <visual>
-	<origin rpy="0 0 0" xyz="0.006625 0 0" />
+	<origin xyz="0 0 -0.01321" />
 	<geometry>
 	  <mesh filename="package://s5fh_controller/description/meshes/f30.dae" />
@@ -227,5 +210,4 @@
     <link name="j">
       <visual>
-	<origin rpy="0 0 0" xyz="0 0 0.02502" />
 	<geometry>
 	  <mesh filename="package://s5fh_controller/description/meshes/f31.dae" />
@@ -236,5 +218,4 @@
     <link name="n">
       <visual>
-	<origin rpy="0 0 0" xyz="0 0 0.01525" />
 	<geometry>
 	  <mesh filename="package://s5fh_controller/description/meshes/f32.dae" />
@@ -245,5 +226,4 @@
     <link name="r">
       <visual>
-	<origin rpy="0 0 0" xyz="0 0 0.00675" />
 	<geometry>
 	  <mesh filename="package://s5fh_controller/description/meshes/f33.dae" />
@@ -255,5 +235,5 @@
     <link name="virtual_i">
       <visual>
-	<origin rpy="0 0 0" xyz="0.02825 0 0" />
+	<origin xyz="0 0 -0.01321" />
 	<geometry>
 	  <mesh filename="package://s5fh_controller/description/meshes/f40.dae" />
@@ -263,5 +243,4 @@
     <link name="i">
       <visual>
-	<origin rpy="0 0 0" xyz="0 0 0.02227" />
 	<geometry>
 	  <mesh filename="package://s5fh_controller/description/meshes/f41.dae" />
@@ -272,5 +251,4 @@
     <link name="m">
       <visual>
-	<origin rpy="0 0 0" xyz="0 0 0.011" />
 	<geometry>
 	  <mesh filename="package://s5fh_controller/description/meshes/f42.dae" />
@@ -281,5 +259,4 @@
     <link name="q">
       <visual>
-	<origin rpy="0 0 0" xyz="0 0 0.0075" />
 	<geometry>
 	  <mesh filename="package://s5fh_controller/description/meshes/f43.dae" />
@@ -289,13 +266,18 @@
     </link>
     <joint name="Thumb_Flexion" type="revolute">
-      <parent link="z" />
+      <parent link="virtual_a" />
       <child link="a" />
       <limit effort="1000.0" lower="0.0" upper="0.9704" velocity="1" />
-      <origin xyz="0 0 0.04596" rpy="0 -1.5707 3.1415" />
-      <axis xyz="0 0 ${side*(1)}" />
+      <origin xyz="0 0 0" rpy="0 0 -0.9704" />
+      <axis xyz="0 0 ${side*(1)}" />
+    </joint>
+    <joint name="Thumb_Helper" type="fixed">
+      <parent link="z" />
+      <child link="virtual_a" />
+      <origin xyz="0 0 0.04596" rpy="0 -1.5707 3.1416" />
     </joint>
     <!-- BASE_LINE JOINTS -->
     <joint name="Thumb_Opposition" type="revolute">
-      <parent link="${name}_base_link" />
+      <parent link="e1" />
       <child link="z" />
       <limit effort="1000.0" lower="0.0" upper="0.9879" velocity="1" />
@@ -305,5 +287,5 @@
     <!-- JOINT NOT FOR BASE_LINE. BUT WRITTEN DOWN HERE FOR BETTER UX -->
     <joint name="f1" type="fixed">
-      <parent link="${name}_base_link" />
+      <parent link="e1" />
       <child link="d" />
       <origin xyz="0 0 0" rpy="0 0 0" />
@@ -322,5 +304,5 @@
       <parent link="${name}_base_link" />
       <child link="e1" />
-      <origin xyz="0 0 0" rpy="0 0 0" />
+      <origin xyz="0 -0.01313 0" rpy="0 0 0" />
     </joint>
     <joint name="j5" type="revolute">
@@ -328,5 +310,5 @@
       <child link="e2" />
       <limit effort="1000.0" lower="0.0" upper="0.98786" velocity="1" />
-      <origin xyz="${side*(0.01840)} 0 0.0375" rpy="0 0 0" />
+      <origin xyz="${side*(0.01840)} 0.006 0.0375" rpy="0 0 0" />
       <axis xyz="0 0 ${side*(1)}" />
       <mimic joint="Thumb_Opposition" multiplier="1" offset="0" />
@@ -335,5 +317,5 @@
       <parent link="e2" />
       <child link="e3" />
-      <origin xyz="0 0 0" rpy="0 0 0" />
+      <origin xyz="0 -0.0060 0" rpy="0 0 0" />
     </joint>
     <joint name="f6" type="fixed">
@@ -481,5 +463,5 @@
       <child link="virtual_j" />
       <limit effort="1000.0" lower="0.0" upper="0.28833" velocity="1" />
-      <origin xyz="${side*(0.00675)} 0 0.0655" rpy="-1.5707 -1.5707 0" />
+      <origin xyz="${side*(0.003855)} 0 0.0655" rpy="-1.5707 -1.5707 0" />
       <axis xyz="0 0 ${side*(1)}" />
       <mimic joint="Finger_Spread" multiplier="0.5" offset="0" />
@@ -489,5 +471,5 @@
       <child link="virtual_i" />
       <limit effort="1000.0" lower="0.0" upper="0.5829" velocity="1" />
-      <origin xyz="${side*(0.02825)} 0 0.056" rpy="-1.5707 -1.5707 0" />
+      <origin xyz="${side*(0.025355)} 0 0.056" rpy="-1.5707 -1.5707 0" />
       <axis xyz="0 0 ${side*(1)}" />
     </joint>

Commit message: remove excess material tags and add proper left hand support

File: s5fh_controller/description/urdf/s5fs.urdf.xacro (robot description, xacro)
@@ -17,34 +17,31 @@
 	  <mesh filename="package://s5fh_controller/description/meshes/base10.dae" />
 	</geometry>
-	<material name="green">
-	  <color rgba="0 1 0 1" />
-	</material>
       </visual>
     </link>
     <link name="d">
-      <visual>
-	<geometry>
-	  <cylinder length="0.110" radius="${cyl_radius}" />
-	</geometry>
-	<material name="green" />
-      </visual>
+      <!-- <visual> -->
+      <!-- 	<geometry> -->
+      <!-- 	  <cylinder length="0.110" radius="${cyl_radius}" /> -->
+      <!-- 	</geometry> -->
+      <!-- 	<material name="green" /> -->
+      <!-- </visual> -->
     </link>
     <link name="h">
-      <visual>
-	<origin rpy="0 1.571 0" xyz="${side*(-0.0125)} 0 0.0825" />
-	<geometry>
-	  <cylinder length="0.025" radius="${cyl_radius}" />
-	</geometry>
-	<material name="green" />
-      </visual>
+      <!-- <visual> -->
+      <!-- 	<origin rpy="0 1.571 0" xyz="${side*(-0.0125)} 0 0.0825" /> -->
+      <!-- 	<geometry> -->
+      <!-- 	  <cylinder length="0.025" radius="${cyl_radius}" /> -->
+      <!-- 	</geometry> -->
+      <!-- 	<material name="green" /> -->
+      <!-- </visual> -->
     </link>
     <link name="d2">
-      <visual>
-	<origin rpy="0 0 0" xyz="${side*(-0.025)} 0 0.09625" />
-	<geometry>
-	  <cylinder length="0.0275" radius="${cyl_radius}" />
-	</geometry>
-	<material name="green" />
-      </visual>
+      <!-- <visual> -->
+      <!-- 	<origin rpy="0 0 0" xyz="${side*(-0.025)} 0 0.09625" /> -->
+      <!-- 	<geometry> -->
+      <!-- 	  <cylinder length="0.0275" radius="${cyl_radius}" /> -->
+      <!-- 	</geometry> -->
+      <!-- 	<material name="green" /> -->
+      <!-- </visual> -->
     </link>
     <!-- LENGTH NOT FOUND IN DATASHEET! GUESSED!!! -->
@@ -53,5 +50,5 @@
 	<origin rpy="0 0 0" xyz="0 0.01313 0" />
 	<geometry>
-	  <mesh filename="package://s5fh_controller/description/meshes/h10.dae" />
+	  <mesh scale="${side*(1)} 1 1" filename="package://s5fh_controller/description/meshes/h10.dae" />
 	</geometry>
       </visual>
@@ -60,7 +57,7 @@
     <link name="e2">
       <visual>
-	<origin xyz="-0.0007 0 -0.01002" />
-	<geometry>
-	  <mesh filename="package://s5fh_controller/description/meshes/h11.dae" />
+	<origin xyz="${side*(-0.0007)} 0 -0.01002" />
+	<geometry>
+	  <mesh scale="${side*(1)} 1 1" filename="package://s5fh_controller/description/meshes/h11.dae" />
 	</geometry>
       </visual>
@@ -68,11 +65,11 @@
     <!-- LENGTH NOT FOUND IN DATASHEET! GUESSED!!! -->
     <link name="e3">
-      <visual>
-	<origin rpy="0 0 0" xyz="${side*(0.0175)} 0 0.015" />
-	<geometry>
-	  <cylinder length="0.03" radius="${cyl_radius}" />
-	</geometry>
-	<material name="green" />
-      </visual>
+      <!-- <visual> -->
+      <!-- 	<origin rpy="0 0 0" xyz="${side*(0.0175)} 0 0.015" /> -->
+      <!-- 	<geometry> -->
+      <!-- 	  <cylinder length="0.03" radius="${cyl_radius}" /> -->
+      <!-- 	</geometry> -->
+      <!-- 	<material name="green" /> -->
+      <!-- </visual> -->
     </link>
     <link name="e">
@@ -80,21 +77,21 @@
     <!-- LENGTH NOT FOUND IN DATASHEET! GUESSED, BUT POSITION CALCULATED: E4 = D-G-F!!! -->
     <link name="e4">
-      <visual>
-	<origin rpy="0 0 0" xyz="${side*(0.02825)} 0 0.043" />
-	<geometry>
-	  <cylinder length="0.026" radius="${cyl_radius}" />
-	</geometry>
-	<material name="green" />
-      </visual>
+      <!-- <visual> -->
+      <!-- 	<origin rpy="0 0 0" xyz="${side*(0.02825)} 0 0.043" /> -->
+      <!-- 	<geometry> -->
+      <!-- 	  <cylinder length="0.026" radius="${cyl_radius}" /> -->
+      <!-- 	</geometry> -->
+      <!-- 	<material name="green" /> -->
+      <!-- </visual> -->
     </link>
     <!-- LENGTH NOT FOUND IN DATASHEET! GUESSED, BUT POSITION CALCULATED: E5 = D-G!!! -->
     <link name="e5">
-      <visual>
-	<origin rpy="0 0 0" xyz="${side*(0.00675)} 0 0.04775" />
-	<geometry>
-	  <cylinder length="0.0355" radius="${cyl_radius}" />
-	</geometry>
-	<material name="green" />
-      </visual>
+      <!-- <visual> -->
+      <!-- 	<origin rpy="0 0 0" xyz="${side*(0.00675)} 0 0.04775" /> -->
+      <!-- 	<geometry> -->
+      <!-- 	  <cylinder length="0.0355" radius="${cyl_radius}" /> -->
+      <!-- 	</geometry> -->
+      <!-- 	<material name="green" /> -->
+      <!-- </visual> -->
     </link>
     <!-- THUMB LINKS -->
@@ -103,7 +100,6 @@
 	<origin xyz="0 0 0.02442" />
 	<geometry>
-	  <mesh filename="package://s5fh_controller/description/meshes/d10.dae" />
-	</geometry>
-	<material name="green" />
+	  <mesh scale="1 ${side*(1)} 1" filename="package://s5fh_controller/description/meshes/d10.dae" />
+	</geometry>
       </visual>
     </link>
@@ -112,7 +108,6 @@
       <visual>
 	<geometry>
-	  <mesh filename="package://s5fh_controller/description/meshes/d11.dae" />
-	</geometry>
-	<material name="green" />
+	  <mesh scale="1 ${side*(1)} ${side*(1)}" filename="package://s5fh_controller/description/meshes/d11.dae" />
+	</geometry>
       </visual>
     </link>
@@ -120,7 +115,6 @@
       <visual>
 	<geometry>
-	  <mesh filename="package://s5fh_controller/description/meshes/d12.dae" />
-	</geometry>
-	<material name="green" />
+	  <mesh scale="1 ${side*(1)} ${side*(1)}" filename="package://s5fh_controller/description/meshes/d12.dae" />
+	</geometry>
       </visual>
     </link>
@@ -128,7 +122,6 @@
       <visual>
 	<geometry>
-	  <mesh filename="package://s5fh_controller/description/meshes/d13.dae" />
-	</geometry>
-	<material name="green" />
+	  <mesh scale="1 ${side*(1)} ${side*(1)}" filename="package://s5fh_controller/description/meshes/d13.dae" />
+	</geometry>
       </visual>
     </link>
@@ -138,5 +131,5 @@
 	<origin xyz="0 0 0.01321" />
 	<geometry>
-	  <mesh filename="package://s5fh_controller/description/meshes/f10.dae" />
+	  <mesh scale="1 ${side*(1)} 1" filename="package://s5fh_controller/description/meshes/f10.dae" />
 	</geometry>
       </visual>
@@ -145,7 +138,6 @@
       <visual>
 	<geometry>
-	  <mesh filename="package://s5fh_controller/description/meshes/f11.dae" />
-	</geometry>
-	<material name="green" />
+	  <mesh scale="1 1 ${side*(1)}" filename="package://s5fh_controller/description/meshes/f11.dae" />
+	</geometry>
       </visual>
     </link>
@@ -153,7 +145,6 @@
       <visual>
 	<geometry>
-	  <mesh filename="package://s5fh_controller/description/meshes/f12.dae" />
-	</geometry>
-	<material name="green" />
+	  <mesh scale="1 1 ${side*(1)}" filename="package://s5fh_controller/description/meshes/f12.dae" />
+	</geometry>
       </visual>
     </link>
@@ -161,7 +152,6 @@
       <visual>
 	<geometry>
-	  <mesh filename="package://s5fh_controller/description/meshes/f13.dae" />
-	</geometry>
-	<material name="green" />
+	  <mesh scale="1 1 ${side*(1)}" filename="package://s5fh_controller/description/meshes/f13.dae" />
+	</geometry>
       </visual>
     </link>
@@ -171,5 +161,5 @@
 	<origin xyz="0 0 0.01321" />
 	<geometry>
-	  <mesh filename="package://s5fh_controller/description/meshes/f20.dae" />
+	  <mesh scale="1 ${side*(1)} 1" filename="package://s5fh_controller/description/meshes/f20.dae" />
 	</geometry>
       </visual>
@@ -178,7 +168,6 @@
       <visual>
 	<geometry>
-	  <mesh filename="package://s5fh_controller/description/meshes/f21.dae" />
-	</geometry>
-	<material name="green" />
+	  <mesh scale="1 1 ${side*(1)}" filename="package://s5fh_controller/description/meshes/f21.dae" />
+	</geometry>
       </visual>
     </link>
@@ -186,7 +175,6 @@
       <visual>
 	<geometry>
-	  <mesh filename="package://s5fh_controller/description/meshes/f22.dae" />
-	</geometry>
-	<material name="green" />
+	  <mesh scale="1 1 ${side*(1)}" filename="package://s5fh_controller/description/meshes/f22.dae" />
+	</geometry>
       </visual>
     </link>
@@ -194,7 +182,6 @@
       <visual>
 	<geometry>
-	  <mesh filename="package://s5fh_controller/description/meshes/f23.dae" />
-	</geometry>
-	<material name="green" />
+	  <mesh scale="1 1 ${side*(1)}" filename="package://s5fh_controller/description/meshes/f23.dae" />
+	</geometry>
       </visual>
     </link>
@@ -204,5 +191,5 @@
 	<origin xyz="0 0 -0.01321" />
 	<geometry>
-	  <mesh filename="package://s5fh_controller/description/meshes/f30.dae" />
+	  <mesh scale="1 ${side*(1)} 1" filename="package://s5fh_controller/description/meshes/f30.dae" />
 	</geometry>
       </visual>
@@ -211,7 +198,6 @@
       <visual>
 	<geometry>
-	  <mesh filename="package://s5fh_controller/description/meshes/f31.dae" />
-	</geometry>
-	<material name="green" />
+	  <mesh scale="1 1 ${side*(1)}" filename="package://s5fh_controller/description/meshes/f31.dae" />
+	</geometry>
       </visual>
     </link>
@@ -219,7 +205,6 @@
       <visual>
 	<geometry>
-	  <mesh filename="package://s5fh_controller/description/meshes/f32.dae" />
-	</geometry>
-	<material name="green" />
+	  <mesh scale="1 1 ${side*(1)}" filename="package://s5fh_controller/description/meshes/f32.dae" />
+	</geometry>
       </visual>
     </link>
@@ -227,7 +212,6 @@
       <visual>
 	<geometry>
-	  <mesh filename="package://s5fh_controller/description/meshes/f33.dae" />
-	</geometry>
-	<material name="green" />
+	  <mesh scale="1 1 ${side*(1)}" filename="package://s5fh_controller/description/meshes/f33.dae" />
+	</geometry>
       </visual>
     </link>
@@ -237,5 +221,5 @@
 	<origin xyz="0 0 -0.01321" />
 	<geometry>
-	  <mesh filename="package://s5fh_controller/description/meshes/f40.dae" />
+	  <mesh scale="1 ${side*(1)} 1" filename="package://s5fh_controller/description/meshes/f40.dae" />
 	</geometry>
       </visual>
@@ -244,7 +228,6 @@
       <visual>
 	<geometry>
-	  <mesh filename="package://s5fh_controller/description/meshes/f41.dae" />
-	</geometry>
-	<material name="green" />
+	  <mesh scale="1 1 ${side*(1)}" filename="package://s5fh_controller/description/meshes/f41.dae" />
+	</geometry>
       </visual>
     </link>
@@ -252,7 +235,6 @@
       <visual>
 	<geometry>
-	  <mesh filename="package://s5fh_controller/description/meshes/f42.dae" />
-	</geometry>
-	<material name="green" />
+	  <mesh scale="1 1 ${side*(1)}" filename="package://s5fh_controller/description/meshes/f42.dae" />
+	</geometry>
       </visual>
     </link>
@@ -260,7 +242,6 @@
       <visual>
 	<geometry>
-	  <mesh filename="package://s5fh_controller/description/meshes/f43.dae" />
-	</geometry>
-	<material name="green" />
+	  <mesh scale="1 1 ${side*(1)}" filename="package://s5fh_controller/description/meshes/f43.dae" />
+	</geometry>
       </visual>
     </link>
@@ -269,5 +250,5 @@
       <child link="a" />
       <limit effort="1000.0" lower="0.0" upper="0.9704" velocity="1" />
-      <origin xyz="0 0 0" rpy="0 0 -0.9704" />
+      <origin xyz="0 0 0" rpy="0 0 ${side*(-0.9704)}" />
       <axis xyz="0 0 ${side*(1)}" />
     </joint>
