Commit message: remove unnecessary scales

File: s5fh_controller/description/urdf/s5fs.urdf.xacro (robot description, xacro)
@@ -131,5 +131,5 @@
 	<origin xyz="0 0 0.01321" />
 	<geometry>
-	  <mesh scale="1 ${side*(1)} 1" filename="package://s5fh_controller/description/meshes/f10.dae" />
+	  <mesh filename="package://s5fh_controller/description/meshes/f10.dae" />
 	</geometry>
       </visual>
@@ -138,5 +138,5 @@
       <visual>
 	<geometry>
-	  <mesh scale="1 1 ${side*(1)}" filename="package://s5fh_controller/description/meshes/f11.dae" />
+	  <mesh filename="package://s5fh_controller/description/meshes/f11.dae" />
 	</geometry>
       </visual>
@@ -145,5 +145,5 @@
       <visual>
 	<geometry>
-	  <mesh scale="1 1 ${side*(1)}" filename="package://s5fh_controller/description/meshes/f12.dae" />
+	  <mesh filename="package://s5fh_controller/description/meshes/f12.dae" />
 	</geometry>
       </visual>
@@ -152,5 +152,5 @@
       <visual>
 	<geometry>
-	  <mesh scale="1 1 ${side*(1)}" filename="package://s5fh_controller/description/meshes/f13.dae" />
+	  <mesh filename="package://s5fh_controller/description/meshes/f13.dae" />
 	</geometry>
       </visual>
@@ -161,5 +161,5 @@
 	<origin xyz="0 0 0.01321" />
 	<geometry>
-	  <mesh scale="1 ${side*(1)} 1" filename="package://s5fh_controller/description/meshes/f20.dae" />
+	  <mesh filename="package://s5fh_controller/description/meshes/f20.dae" />
 	</geometry>
       </visual>
@@ -168,5 +168,5 @@
       <visual>
 	<geometry>
-	  <mesh scale="1 1 ${side*(1)}" filename="package://s5fh_controller/description/meshes/f21.dae" />
+	  <mesh filename="package://s5fh_controller/description/meshes/f21.dae" />
 	</geometry>
       </visual>
@@ -175,5 +175,5 @@
       <visual>
 	<geometry>
-	  <mesh scale="1 1 ${side*(1)}" filename="package://s5fh_controller/description/meshes/f22.dae" />
+	  <mesh filename="package://s5fh_controller/description/meshes/f22.dae" />
 	</geometry>
       </visual>
@@ -182,5 +182,5 @@
       <visual>
 	<geometry>
-	  <mesh scale="1 1 ${side*(1)}" filename="package://s5fh_controller/description/meshes/f23.dae" />
+	  <mesh filename="package://s5fh_controller/description/meshes/f23.dae" />
 	</geometry>
       </visual>
@@ -191,5 +191,5 @@
 	<origin xyz="0 0 -0.01321" />
 	<geometry>
-	  <mesh scale="1 ${side*(1)} 1" filename="package://s5fh_controller/description/meshes/f30.dae" />
+	  <mesh filename="package://s5fh_controller/description/meshes/f30.dae" />
 	</geometry>
       </visual>
@@ -198,5 +198,5 @@
       <visual>
 	<geometry>
-	  <mesh scale="1 1 ${side*(1)}" filename="package://s5fh_controller/description/meshes/f31.dae" />
+	  <mesh filename="package://s5fh_controller/description/meshes/f31.dae" />
 	</geometry>
       </visual>
@@ -205,5 +205,5 @@
       <visual>
 	<geometry>
-	  <mesh scale="1 1 ${side*(1)}" filename="package://s5fh_controller/description/meshes/f32.dae" />
+	  <mesh filename="package://s5fh_controller/description/meshes/f32.dae" />
 	</geometry>
       </visual>
@@ -212,5 +212,5 @@
       <visual>
 	<geometry>
-	  <mesh scale="1 1 ${side*(1)}" filename="package://s5fh_controller/description/meshes/f33.dae" />
+	  <mesh filename="package://s5fh_controller/description/meshes/f33.dae" />
 	</geometry>
       </visual>
@@ -221,5 +221,5 @@
 	<origin xyz="0 0 -0.01321" />
 	<geometry>
-	  <mesh scale="1 ${side*(1)} 1" filename="package://s5fh_controller/description/meshes/f40.dae" />
+	  <mesh filename="package://s5fh_controller/description/meshes/f40.dae" />
 	</geometry>
       </visual>
@@ -228,5 +228,5 @@
       <visual>
 	<geometry>
-	  <mesh scale="1 1 ${side*(1)}" filename="package://s5fh_controller/description/meshes/f41.dae" />
+	  <mesh filename="package://s5fh_controller/description/meshes/f41.dae" />
 	</geometry>
       </visual>
@@ -235,5 +235,5 @@
       <visual>
 	<geometry>
-	  <mesh scale="1 1 ${side*(1)}" filename="package://s5fh_controller/description/meshes/f42.dae" />
+	  <mesh filename="package://s5fh_controller/description/meshes/f42.dae" />
 	</geometry>
       </visual>
@@ -242,5 +242,5 @@
       <visual>
 	<geometry>
-	  <mesh scale="1 1 ${side*(1)}" filename="package://s5fh_controller/description/meshes/f43.dae" />
+	  <mesh filename="package://s5fh_controller/description/meshes/f43.dae" />
 	</geometry>
       </visual>
