Commit message: Changed a slight error in multiplication factor.

File: description/urdf/s5fs.urdf.xacro (robot description, xacro)
@@ -377,5 +377,5 @@
       <origin xyz="0.032 0 0" rpy="0 0 0" />
       <axis xyz="0 0 1" />
-      <mimic joint="Middle_Finger_Distal" multiplier="1.000" offset="0" />
+      <mimic joint="Middle_Finger_Distal" multiplier="1.0454" offset="0" />
     </joint>
     <!-- RING FINGER JOINTS -->
