Commit message: Renamed the descriptions as well (untestet). Package name is now svh_driver

File: description/urdf/svh-arm.urdf.xacro (robot description, xacro)
@@ -1,4 +1,4 @@
 <?xml version="1.0"?>
-<robot name="s5fs-arm" xmlns:xacro="http://www.ros.org/wiki/xacro">
+<robot name="svh-arm" xmlns:xacro="http://www.ros.org/wiki/xacro">
    <material name="Schunk/Blue">
     <color rgba="0.6 0.6 0.6 1"/>
@@ -7,5 +7,5 @@
     <color rgba="0 0 .8 1"/>
   </material>
- <xacro:include filename="$(find s5fh_controller)/description/urdf/s5fs.urdf.xacro" />
+ <xacro:include filename="$(find svh_controller)/description/urdf/svh.urdf.xacro" />
  <xacro:include filename="$(find schunk_description)/urdf/lwa4p/lwa4p.urdf.xacro" />
  <link name="base_link" />
@@ -19,6 +19,6 @@
       <xacro:property name="arm_6_ref" value="2.1" />
   </xacro:schunk_lwa4p>
- <xacro:s5fh parent="arm_6_link" name="left_hand" side="-1">
+ <xacro:svh parent="arm_6_link" name="left_hand" side="-1">
     <origin xyz="0 0 0.1"  rpy= "0 0 0" />
-  </xacro:s5fh>
+  </xacro:svh>
 </robot>

File: description/urdf/svh.urdf.xacro (robot description, xacro)
@@ -2,5 +2,5 @@
 <robot xmlns:xacro="http://www.ros.org/wiki/xacro">
   <xacro:property name="cyl_radius" value="0.001" />
-  <xacro:macro name="s5fh" params="parent name side *origin">
+  <xacro:macro name="svh" params="parent name side *origin">
     <!-- RIGHT HAND = 1, LEFT HAND = -1 -->
     <!-- BASE_LINE LINKS -->
@@ -15,5 +15,5 @@
 	<origin xyz="0 0 -0.032" rpy="0 0 0" />
 	<geometry>
-	  <mesh filename="package://s5fh_controller/description/meshes/base10.dae" />
+	  <mesh filename="package://svh_controller/description/meshes/base10.dae" />
 	</geometry>
       </visual>
@@ -50,5 +50,5 @@
 	<origin rpy="0 0 0" xyz="0 0.01313 0" />
 	<geometry>
-	  <mesh scale="${side*(1)} 1 1" filename="package://s5fh_controller/description/meshes/h10.dae" />
+	  <mesh scale="${side*(1)} 1 1" filename="package://svh_controller/description/meshes/h10.dae" />
 	</geometry>
       </visual>
@@ -59,5 +59,5 @@
 	<origin xyz="${side*(-0.0007)} 0 -0.01002" />
 	<geometry>
-	  <mesh scale="${side*(1)} 1 1" filename="package://s5fh_controller/description/meshes/h11.dae" />
+	  <mesh scale="${side*(1)} 1 1" filename="package://svh_controller/description/meshes/h11.dae" />
 	</geometry>
       </visual>
@@ -100,5 +100,5 @@
 	<origin xyz="0 0 0.02442" />
 	<geometry>
-	  <mesh scale="1 ${side*(1)} 1" filename="package://s5fh_controller/description/meshes/d10.dae" />
+	  <mesh scale="1 ${side*(1)} 1" filename="package://svh_controller/description/meshes/d10.dae" />
 	</geometry>
       </visual>
@@ -108,5 +108,5 @@
       <visual>
 	<geometry>
-	  <mesh scale="1 ${side*(1)} ${side*(1)}" filename="package://s5fh_controller/description/meshes/d11.dae" />
+	  <mesh scale="1 ${side*(1)} ${side*(1)}" filename="package://svh_controller/description/meshes/d11.dae" />
 	</geometry>
       </visual>
@@ -115,5 +115,5 @@
       <visual>
 	<geometry>
-	  <mesh scale="1 ${side*(1)} ${side*(1)}" filename="package://s5fh_controller/description/meshes/d12.dae" />
+	  <mesh scale="1 ${side*(1)} ${side*(1)}" filename="package://svh_controller/description/meshes/d12.dae" />
 	</geometry>
       </visual>
@@ -122,5 +122,5 @@
       <visual>
 	<geometry>
-	  <mesh scale="1 ${side*(1)} ${side*(1)}" filename="package://s5fh_controller/description/meshes/d13.dae" />
+	  <mesh scale="1 ${side*(1)} ${side*(1)}" filename="package://svh_controller/description/meshes/d13.dae" />
 	</geometry>
       </visual>
@@ -131,5 +131,5 @@
 	<origin xyz="0 0 0.01321" />
 	<geometry>
-	  <mesh filename="package://s5fh_controller/description/meshes/f10.dae" />
+	  <mesh filename="package://svh_controller/description/meshes/f10.dae" />
 	</geometry>
       </visual>
@@ -138,5 +138,5 @@
       <visual>
 	<geometry>
-	  <mesh filename="package://s5fh_controller/description/meshes/f11.dae" />
+	  <mesh filename="package://svh_controller/description/meshes/f11.dae" />
 	</geometry>
       </visual>
@@ -145,5 +145,5 @@
       <visual>
 	<geometry>
-	  <mesh filename="package://s5fh_controller/description/meshes/f12.dae" />
+	  <mesh filename="package://svh_controller/description/meshes/f12.dae" />
 	</geometry>
       </visual>
@@ -152,5 +152,5 @@
       <visual>
 	<geometry>
-	  <mesh filename="package://s5fh_controller/description/meshes/f13.dae" />
+	  <mesh filename="package://svh_controller/description/meshes/f13.dae" />
 	</geometry>
       </visual>
@@ -161,5 +161,5 @@
 	<origin xyz="0 0 0.01321" />
 	<geometry>
-	  <mesh filename="package://s5fh_controller/description/meshes/f20.dae" />
+	  <mesh filename="package://svh_controller/description/meshes/f20.dae" />
 	</geometry>
       </visual>
@@ -168,5 +168,5 @@
       <visual>
 	<geometry>
-	  <mesh filename="package://s5fh_controller/description/meshes/f21.dae" />
+	  <mesh filename="package://svh_controller/description/meshes/f21.dae" />
 	</geometry>
       </visual>
@@ -175,5 +175,5 @@
       <visual>
 	<geometry>
-	  <mesh filename="package://s5fh_controller/description/meshes/f22.dae" />
+	  <mesh filename="package://svh_controller/description/meshes/f22.dae" />
 	</geometry>
       </visual>
@@ -182,5 +182,5 @@
       <visual>
 	<geometry>
-	  <mesh filename="package://s5fh_controller/description/meshes/f23.dae" />
+	  <mesh filename="package://svh_controller/description/meshes/f23.dae" />
 	</geometry>
       </visual>
@@ -191,5 +191,5 @@
 	<origin xyz="0 0 -0.01321" />
 	<geometry>
-	  <mesh filename="package://s5fh_controller/description/meshes/f30.dae" />
+	  <mesh filename="package://svh_controller/description/meshes/f30.dae" />
 	</geometry>
       </visual>
@@ -198,5 +198,5 @@
       <visual>
 	<geometry>
-	  <mesh filename="package://s5fh_controller/description/meshes/f31.dae" />
+	  <mesh filename="package://svh_controller/description/meshes/f31.dae" />
 	</geometry>
       </visual>
@@ -205,5 +205,5 @@
       <visual>
 	<geometry>
-	  <mesh filename="package://s5fh_controller/description/meshes/f32.dae" />
+	  <mesh filename="package://svh_controller/description/meshes/f32.dae" />
 	</geometry>
       </visual>
@@ -212,5 +212,5 @@
       <visual>
 	<geometry>
-	  <mesh filename="package://s5fh_controller/description/meshes/f33.dae" />
+	  <mesh filename="package://svh_controller/description/meshes/f33.dae" />
 	</geometry>
       </visual>
@@ -221,5 +221,5 @@
 	<origin xyz="0 0 -0.01321" />
 	<geometry>
-	  <mesh filename="package://s5fh_controller/description/meshes/f40.dae" />
+	  <mesh filename="package://svh_controller/description/meshes/f40.dae" />
 	</geometry>
       </visual>
@@ -228,5 +228,5 @@
       <visual>
 	<geometry>
-	  <mesh filename="package://s5fh_controller/description/meshes/f41.dae" />
+	  <mesh filename="package://svh_controller/description/meshes/f41.dae" />
 	</geometry>
       </visual>
@@ -235,5 +235,5 @@
       <visual>
 	<geometry>
-	  <mesh filename="package://s5fh_controller/description/meshes/f42.dae" />
+	  <mesh filename="package://svh_controller/description/meshes/f42.dae" />
 	</geometry>
       </visual>
@@ -242,5 +242,5 @@
       <visual>
 	<geometry>
-	  <mesh filename="package://s5fh_controller/description/meshes/f43.dae" />
+	  <mesh filename="package://svh_controller/description/meshes/f43.dae" />
 	</geometry>
       </visual>
