Commit message: Make hand member names dependent of hand name

File: description/urdf/svh.urdf.xacro (robot description, xacro)
@@ -19,82 +19,82 @@
       </visual>
     </link>
-    <link name="d">
+    <link name="${name}_d">
       <!-- <visual> -->
       <!-- 	<geometry> -->
       <!-- 	  <cylinder length="0.110" radius="${cyl_radius}" /> -->
       <!-- 	</geometry> -->
+      <!-- 	<material name="${name}_green" /> -->
+      <!-- </visual> -->
+    </link>
+    <link name="${name}_h">
+      <!-- <visual> -->
+      <!-- 	<origin rpy="0 1.571 0" xyz="${side*(-0.0125)} 0 0.0825" /> -->
+      <!-- 	<geometry> -->
+      <!-- 	  <cylinder length="0.025" radius="${cyl_radius}" /> -->
+      <!-- 	</geometry> -->
+      <!-- 	<material name="${name}_green" /> -->
+      <!-- </visual> -->
+    </link>
+    <link name="${name}_d2">
+      <!-- <visual> -->
+      <!-- 	<origin rpy="0 0 0" xyz="${side*(-0.025)} 0 0.09625" /> -->
+      <!-- 	<geometry> -->
+      <!-- 	  <cylinder length="0.0275" radius="${cyl_radius}" /> -->
+      <!-- 	</geometry> -->
+      <!-- 	<material name="${name}_green" /> -->
+      <!-- </visual> -->
+    </link>
+    <!-- LENGTH NOT FOUND IN DATASHEET! GUESSED!!! -->
+    <link name="${name}_e1">
+      <visual>
+	<origin rpy="0 0 0" xyz="0 0.01313 0" />
+	<geometry>
+          <mesh scale="${side*(1)} 1 1" filename="package://schunk_svh_driver/description/meshes/h10.dae" />
+	</geometry>
+      </visual>
+    </link>
+    <!-- LENGTH NOT FOUND IN DATASHEET! GUESSED!!! -->
+    <link name="${name}_e2">
+      <visual>
+	<origin xyz="${side*(-0.0007)} 0 -0.01002" />
+	<geometry>
+          <mesh scale="${side*(1)} 1 1" filename="package://schunk_svh_driver/description/meshes/h11.dae" />
+	</geometry>
+      </visual>
+    </link>
+    <!-- LENGTH NOT FOUND IN DATASHEET! GUESSED!!! -->
+    <link name="${name}_e3">
+      <!-- <visual> -->
+      <!-- 	<origin rpy="0 0 0" xyz="${side*(0.0175)} 0 0.015" /> -->
+      <!-- 	<geometry> -->
+      <!-- 	  <cylinder length="0.03" radius="${cyl_radius}" /> -->
+      <!-- 	</geometry> -->
       <!-- 	<material name="green" /> -->
       <!-- </visual> -->
     </link>
-    <link name="h">
-      <!-- <visual> -->
-      <!-- 	<origin rpy="0 1.571 0" xyz="${side*(-0.0125)} 0 0.0825" /> -->
-      <!-- 	<geometry> -->
-      <!-- 	  <cylinder length="0.025" radius="${cyl_radius}" /> -->
+    <link name="${name}_e">
+    </link>
+    <!-- LENGTH NOT FOUND IN DATASHEET! GUESSED, BUT POSITION CALCULATED: E4 = D-G-F!!! -->
+    <link name="${name}_e4">
+      <!-- <visual> -->
+      <!-- 	<origin rpy="0 0 0" xyz="${side*(0.02825)} 0 0.043" /> -->
+      <!-- 	<geometry> -->
+      <!-- 	  <cylinder length="0.026" radius="${cyl_radius}" /> -->
       <!-- 	</geometry> -->
       <!-- 	<material name="green" /> -->
       <!-- </visual> -->
     </link>
-    <link name="d2">
-      <!-- <visual> -->
-      <!-- 	<origin rpy="0 0 0" xyz="${side*(-0.025)} 0 0.09625" /> -->
-      <!-- 	<geometry> -->
-      <!-- 	  <cylinder length="0.0275" radius="${cyl_radius}" /> -->
+    <!-- LENGTH NOT FOUND IN DATASHEET! GUESSED, BUT POSITION CALCULATED: E5 = D-G!!! -->
+    <link name="${name}_e5">
+      <!-- <visual> -->
+      <!-- 	<origin rpy="0 0 0" xyz="${side*(0.00675)} 0 0.04775" /> -->
+      <!-- 	<geometry> -->
+      <!-- 	  <cylinder length="0.0355" radius="${cyl_radius}" /> -->
       <!-- 	</geometry> -->
       <!-- 	<material name="green" /> -->
       <!-- </visual> -->
     </link>
-    <!-- LENGTH NOT FOUND IN DATASHEET! GUESSED!!! -->
-    <link name="e1">
-      <visual>
-	<origin rpy="0 0 0" xyz="0 0.01313 0" />
-	<geometry>
-          <mesh scale="${side*(1)} 1 1" filename="package://schunk_svh_driver/description/meshes/h10.dae" />
-	</geometry>
-      </visual>
-    </link>
-    <!-- LENGTH NOT FOUND IN DATASHEET! GUESSED!!! -->
-    <link name="e2">
-      <visual>
-	<origin xyz="${side*(-0.0007)} 0 -0.01002" />
-	<geometry>
-          <mesh scale="${side*(1)} 1 1" filename="package://schunk_svh_driver/description/meshes/h11.dae" />
-	</geometry>
-      </visual>
-    </link>
-    <!-- LENGTH NOT FOUND IN DATASHEET! GUESSED!!! -->
-    <link name="e3">
-      <!-- <visual> -->
-      <!-- 	<origin rpy="0 0 0" xyz="${side*(0.0175)} 0 0.015" /> -->
-      <!-- 	<geometry> -->
-      <!-- 	  <cylinder length="0.03" radius="${cyl_radius}" /> -->
-      <!-- 	</geometry> -->
-      <!-- 	<material name="green" /> -->
-      <!-- </visual> -->
-    </link>
-    <link name="e">
-    </link>
-    <!-- LENGTH NOT FOUND IN DATASHEET! GUESSED, BUT POSITION CALCULATED: E4 = D-G-F!!! -->
-    <link name="e4">
-      <!-- <visual> -->
-      <!-- 	<origin rpy="0 0 0" xyz="${side*(0.02825)} 0 0.043" /> -->
-      <!-- 	<geometry> -->
-      <!-- 	  <cylinder length="0.026" radius="${cyl_radius}" /> -->
-      <!-- 	</geometry> -->
-      <!-- 	<material name="green" /> -->
-      <!-- </visual> -->
-    </link>
-    <!-- LENGTH NOT FOUND IN DATASHEET! GUESSED, BUT POSITION CALCULATED: E5 = D-G!!! -->
-    <link name="e5">
-      <!-- <visual> -->
-      <!-- 	<origin rpy="0 0 0" xyz="${side*(0.00675)} 0 0.04775" /> -->
-      <!-- 	<geometry> -->
-      <!-- 	  <cylinder length="0.0355" radius="${cyl_radius}" /> -->
-      <!-- 	</geometry> -->
-      <!-- 	<material name="green" /> -->
-      <!-- </visual> -->
-    </link>
     <!-- THUMB LINKS -->
-    <link name="z">
+    <link name="${name}_z">
       <visual>
 	<origin xyz="0 0 0.02442" />
@@ -104,6 +104,6 @@
       </visual>
     </link>
-    <link name="virtual_a" />
-    <link name="a">
+    <link name="${name}_virtual_a" />
+    <link name="${name}_a">
       <visual>
 	<geometry>
@@ -112,5 +112,5 @@
       </visual>
     </link>
-    <link name="b">
+    <link name="${name}_b">
       <visual>
 	<geometry>
@@ -119,5 +119,5 @@
       </visual>
     </link>
-    <link name="c">
+    <link name="${name}_c">
       <visual>
 	<geometry>
@@ -127,5 +127,5 @@
     </link>
     <!-- INDEX FINGER LINKS -->
-    <link name="virtual_l">
+    <link name="${name}_virtual_l">
       <visual>
 	<origin xyz="0 0 0.01321" />
@@ -135,5 +135,5 @@
       </visual>
     </link>
-    <link name="l">
+    <link name="${name}_l">
       <visual>
 	<geometry>
@@ -142,5 +142,5 @@
       </visual>
     </link>
-    <link name="p">
+    <link name="${name}_p">
       <visual>
 	<geometry>
@@ -149,5 +149,5 @@
       </visual>
     </link>
-    <link name="t">
+    <link name="${name}_t">
       <visual>
 	<geometry>
@@ -157,5 +157,5 @@
     </link>
     <!-- MIDDLE FINGER LINKS -->
-    <link name="virtual_k">
+    <link name="${name}_virtual_k">
       <visual>
 	<origin xyz="0 0 0.01321" />
@@ -165,5 +165,5 @@
       </visual>
     </link>
-    <link name="k">
+    <link name="${name}_k">
       <visual>
 	<geometry>
@@ -172,5 +172,5 @@
       </visual>
     </link>
-    <link name="o">
+    <link name="${name}_o">
       <visual>
 	<geometry>
@@ -179,5 +179,5 @@
       </visual>
     </link>
-    <link name="s">
+    <link name="${name}_s">
       <visual>
 	<geometry>
@@ -187,5 +187,5 @@
     </link>
     <!-- RING FINGER LINKS -->
-    <link name="virtual_j">
+    <link name="${name}_virtual_j">
       <visual>
 	<origin xyz="0 0 -0.01321" />
@@ -195,5 +195,5 @@
       </visual>
     </link>
-    <link name="j">
+    <link name="${name}_j">
       <visual>
 	<geometry>
@@ -202,5 +202,5 @@
       </visual>
     </link>
-    <link name="n">
+    <link name="${name}_n">
       <visual>
 	<geometry>
@@ -209,5 +209,5 @@
       </visual>
     </link>
-    <link name="r">
+    <link name="${name}_r">
       <visual>
 	<geometry>
@@ -217,5 +217,5 @@
     </link>
     <!-- LITTLE FINGER LINKS -->
-    <link name="virtual_i">
+    <link name="${name}_virtual_i">
       <visual>
 	<origin xyz="0 0 -0.01321" />
@@ -225,5 +225,5 @@
       </visual>
     </link>
-    <link name="i">
+    <link name="${name}_i">
       <visual>
 	<geometry>
@@ -232,5 +232,5 @@
       </visual>
     </link>
-    <link name="m">
+    <link name="${name}_m">
       <visual>
 	<geometry>
@@ -239,5 +239,5 @@
       </visual>
     </link>
-    <link name="q">
+    <link name="${name}_q">
       <visual>
 	<geometry>
@@ -246,20 +246,20 @@
       </visual>
     </link>
-    <joint name="Thumb_Flexion" type="revolute">
-      <parent link="virtual_a" />
-      <child link="a" />
+    <joint name="${name}_Thumb_Flexion" type="revolute">
+      <parent link="${name}_virtual_a" />
+      <child link="${name}_a" />
       <limit effort="1000.0" lower="0.0" upper="0.9704" velocity="1" />
       <origin xyz="0 0 0" rpy="0 0 ${side*(-0.9704)}" />
       <axis xyz="0 0 ${side*(1)}" />
     </joint>
-    <joint name="Thumb_Helper" type="fixed">
-      <parent link="z" />
-      <child link="virtual_a" />
+    <joint name="${name}_Thumb_Helper" type="fixed">
+      <parent link="${name}_z" />
+      <child link="${name}_virtual_a" />
       <origin xyz="0 0 0.04596" rpy="0 -1.5707 3.1416" />
     </joint>
     <!-- BASE_LINE JOINTS -->
-    <joint name="Thumb_Opposition" type="revolute">
-      <parent link="e1" />
-      <child link="z" />
+    <joint name="${name}_Thumb_Opposition" type="revolute">
+      <parent link="${name}_e1" />
+      <child link="${name}_z" />
       <limit effort="1000.0" lower="0.0" upper="0.9879" velocity="1" />
       <origin xyz="${side*(-0.01690)} 0.02626 0" rpy="0 0.2618 1.571" />
@@ -267,27 +267,27 @@
     </joint>
     <!-- JOINT NOT FOR BASE_LINE. BUT WRITTEN DOWN HERE FOR BETTER UX -->
-    <joint name="f1" type="fixed">
-      <parent link="e1" />
-      <child link="d" />
-      <origin xyz="0 0 0" rpy="0 0 0" />
-    </joint>
-    <joint name="f2" type="fixed">
-      <parent link="d" />
-      <child link="h" />
-      <origin xyz="0 0 0" rpy="0 0 0" />
-    </joint>
-    <joint name="f3" type="fixed">
-      <parent link="h" />
-      <child link="d2" />
-      <origin xyz="0 0 0" rpy="0 0 0" />
-    </joint>
-    <joint name="f4" type="fixed">
+    <joint name="${name}_f1" type="fixed">
+      <parent link="${name}_e1" />
+      <child link="${name}_d" />
+      <origin xyz="0 0 0" rpy="0 0 0" />
+    </joint>
+    <joint name="${name}_f2" type="fixed">
+      <parent link="${name}_d" />
+      <child link="${name}_h" />
+      <origin xyz="0 0 0" rpy="0 0 0" />
+    </joint>
+    <joint name="${name}_f3" type="fixed">
+      <parent link="${name}_h" />
+      <child link="${name}_d2" />
+      <origin xyz="0 0 0" rpy="0 0 0" />
+    </joint>
+    <joint name="${name}_f4" type="fixed">
       <parent link="${name}_base_link" />
-      <child link="e1" />
+      <child link="${name}_e1" />
       <origin xyz="0 -0.01313 0" rpy="0 0 0" />
     </joint>
-    <joint name="j5" type="revolute">
-      <parent link="e1" />
-      <child link="e2" />
+    <joint name="${name}_j5" type="revolute">
+      <parent link="${name}_e1" />
+      <child link="${name}_e2" />
       <limit effort="1000.0" lower="0.0" upper="0.98786" velocity="1" />
       <origin xyz="${side*(0.01840)} 0.006 0.0375" rpy="0 0 0" />
@@ -295,28 +295,28 @@
       <mimic joint="Thumb_Opposition" multiplier="1" offset="0" />
     </joint>
-    <joint name="f5" type="fixed">
-      <parent link="e2" />
-      <child link="e3" />
+    <joint name="${name}_f5" type="fixed">
+      <parent link="${name}_e2" />
+      <child link="${name}_e3" />
       <origin xyz="0 -0.0060 0" rpy="0 0 0" />
     </joint>
-    <joint name="f6" type="fixed">
-      <parent link="e3" />
-      <child link="e" />
-      <origin xyz="0 0 0" rpy="0 0 0" />
-    </joint>
-    <joint name="f7" type="fixed">
-      <parent link="e" />
-      <child link="e4" />
-      <origin xyz="0 0 0" rpy="0 0 0" />
-    </joint>
-    <joint name="f8" type="fixed">
-      <parent link="e" />
-      <child link="e5" />
+    <joint name="${name}_f6" type="fixed">
+      <parent link="${name}_e3" />
+      <child link="${name}_e" />
+      <origin xyz="0 0 0" rpy="0 0 0" />
+    </joint>
+    <joint name="${name}_f7" type="fixed">
+      <parent link="${name}_e" />
+      <child link="${name}_e4" />
+      <origin xyz="0 0 0" rpy="0 0 0" />
+    </joint>
+    <joint name="${name}_f8" type="fixed">
+      <parent link="${name}_e" />
+      <child link="${name}_e5" />
       <origin xyz="0 0 0" rpy="0 0 0" />
     </joint>
     <!-- THUMB JOINTS -->
-    <joint name="j3" type="revolute">
-      <parent link="a" />
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
Commit message: Added a name prefix to allow multiple instantiation of the hand model.

File: description/urdf/svh.urdf.xacro (robot description, xacro)
@@ -293,5 +293,5 @@
       <origin xyz="${side*(0.01840)} 0.006 0.0375" rpy="0 0 0" />
       <axis xyz="0 0 ${side*(1)}" />
-      <mimic joint="Thumb_Opposition" multiplier="1" offset="0" />
+      <mimic joint="${name}_Thumb_Opposition" multiplier="1" offset="0" />
     </joint>
     <joint name="${name}_f5" type="fixed">
@@ -322,5 +322,5 @@
       <origin xyz="0.0485 0 0" rpy="0 0 0" />
       <axis xyz="0 0 ${side*(1)}" />
-      <mimic joint="Thumb_Flexion" multiplier="1.01511" offset="0" />
+      <mimic joint="${name}_Thumb_Flexion" multiplier="1.01511" offset="0" />
     </joint>
     <joint name="${name}_j4" type="revolute">
@@ -330,5 +330,5 @@
       <origin xyz="0.030 0 0" rpy="0 0 0" />
       <axis xyz="0 0 ${side*(1)}" />
-      <mimic joint="Thumb_Flexion" multiplier="1.44889" offset="0" />
+      <mimic joint="${name}_Thumb_Flexion" multiplier="1.44889" offset="0" />
     </joint>
     <!-- INDEX FINGER JOINTS -->
@@ -354,5 +354,5 @@
       <origin xyz="0.026 0 0" rpy="0 0 0" />
       <axis xyz="0 0 1" />
-      <mimic joint="Index_Finger_Distal" multiplier="1.0450" offset="0" />
+      <mimic joint="${name}_Index_Finger_Distal" multiplier="1.0450" offset="0" />
     </joint>
     <!-- MIDDLE FINGER JOINTS -->
@@ -377,5 +377,5 @@
       <origin xyz="0.032 0 0" rpy="0 0 0" />
       <axis xyz="0 0 1" />
-      <mimic joint="Middle_Finger_Distal" multiplier="1.0454" offset="0" />
+      <mimic joint="${name}_Middle_Finger_Distal" multiplier="1.0454" offset="0" />
     </joint>
     <!-- RING FINGER JOINTS -->
@@ -393,5 +393,5 @@
       <origin xyz="0.05004 0 0" rpy="0 0 0" />
       <axis xyz="0 0 1" />
-      <mimic joint="Ring_Finger" multiplier="1.3588" offset="0" />
+      <mimic joint="${name}_Ring_Finger" multiplier="1.3588" offset="0" />
     </joint>
     <joint name="${name}_j16" type="revolute">
@@ -401,5 +401,5 @@
       <origin xyz="0.032 0 0" rpy="0 0 0" />
       <axis xyz="0 0 1" />
-      <mimic joint="Ring_Finger" multiplier="1.42093" offset="0" />
+      <mimic joint="${name}_Ring_Finger" multiplier="1.42093" offset="0" />
     </joint>
     <!-- PINKY JOINTS -->
@@ -417,5 +417,5 @@
       <origin xyz="0.04454 0 0" rpy="0 0 0" />
       <axis xyz="0 0 1" />
-      <mimic joint="Pinky" multiplier="1.35880" offset="0" />
+      <mimic joint="${name}_Pinky" multiplier="1.35880" offset="0" />
     </joint>
     <joint name="${name}_j17" type="revolute">
@@ -425,5 +425,5 @@
       <origin xyz="0.022 0 0" rpy="0 0 0" />
       <axis xyz="0 0 1" />
-      <mimic joint="Pinky" multiplier="1.42307" offset="0" />
+      <mimic joint="${name}_Pinky" multiplier="1.42307" offset="0" />
     </joint>
     <joint name="${name}_index_spread" type="revolute">
@@ -433,5 +433,5 @@
       <origin xyz="${side*(-0.025)} 0 0.110" rpy="0 -1.5707 1.5707" />
       <axis xyz="0 0 ${side*(1)}" />
-      <mimic joint="Finger_Spread" multiplier="0.5" offset="0" />
+      <mimic joint="${name}_Finger_Spread" multiplier="0.5" offset="0" />
     </joint>
     <joint name="${name}_middle_spread_dummy" type="fixed">
@@ -446,5 +446,5 @@
       <origin xyz="${side*(0.003855)} 0 0.0655" rpy="-1.5707 -1.5707 0" />
       <axis xyz="0 0 ${side*(1)}" />
-      <mimic joint="Finger_Spread" multiplier="0.5" offset="0" />
+      <mimic joint="${name}_Finger_Spread" multiplier="0.5" offset="0" />
     </joint>
     <joint name="${name}_Finger_Spread" type="revolute">

Commit message: add collision meshes to URDF

File: description/urdf/svh.urdf.xacro (robot description, xacro)
@@ -18,4 +18,10 @@
 	</geometry>
       </visual>
+      <collision>
+	<origin xyz="0 0 -0.032" rpy="0 0 0" />
+	<geometry>
+          <mesh filename="package://schunk_svh_driver/description/meshes/base10.dae" />
+	</geometry>
+      </collision>
     </link>
     <link name="${name}_d">
@@ -53,4 +59,10 @@
 	</geometry>
       </visual>
+      <collision>
+	<origin rpy="0 0 0" xyz="0 0.01313 0" />
+	<geometry>
+          <mesh scale="${side*(1)} 1 1" filename="package://schunk_svh_driver/description/meshes/h10.dae" />
+	</geometry>
+      </collision>
     </link>
     <!-- LENGTH NOT FOUND IN DATASHEET! GUESSED!!! -->
@@ -62,4 +74,10 @@
 	</geometry>
       </visual>
+      <collision>
+	<origin xyz="${side*(-0.0007)} 0 -0.01002" />
+	<geometry>
+          <mesh scale="${side*(1)} 1 1" filename="package://schunk_svh_driver/description/meshes/h11.dae" />
+	</geometry>
+      </collision>
     </link>
     <!-- LENGTH NOT FOUND IN DATASHEET! GUESSED!!! -->
@@ -103,4 +121,10 @@
 	</geometry>
       </visual>
+      <collision>
+	<origin xyz="0 0 0.02442" />
+	<geometry>
+          <mesh scale="1 ${side*(1)} 1" filename="package://schunk_svh_driver/description/meshes/d10.dae" />
+	</geometry>
+      </collision>
     </link>
     <link name="${name}_virtual_a" />
@@ -111,4 +135,9 @@
 	</geometry>
       </visual>
+      <collision>
+	<geometry>
+          <mesh scale="1 ${side*(1)} ${side*(1)}" filename="package://schunk_svh_driver/description/meshes/d11.dae" />
+	</geometry>
+      </collision>
     </link>
     <link name="${name}_b">
@@ -118,4 +147,9 @@
 	</geometry>
       </visual>
+      <collision>
+	<geometry>
+          <mesh scale="1 ${side*(1)} ${side*(1)}" filename="package://schunk_svh_driver/description/meshes/d12.dae" />
+	</geometry>
+      </collision>
     </link>
     <link name="${name}_c">
@@ -125,4 +159,9 @@
 	</geometry>
       </visual>
+      <collision>
+	<geometry>
+          <mesh scale="1 ${side*(1)} ${side*(1)}" filename="package://schunk_svh_driver/description/meshes/d13.dae" />
+	</geometry>
+      </collision>
     </link>
     <!-- INDEX FINGER LINKS -->
@@ -134,4 +173,10 @@
 	</geometry>
       </visual>
+      <collision>
+	<origin xyz="0 0 0.01321" />
+	<geometry>
+          <mesh filename="package://schunk_svh_driver/description/meshes/f10.dae" />
+	</geometry>
+      </collision>
     </link>
     <link name="${name}_l">
@@ -141,4 +186,9 @@
 	</geometry>
       </visual>
+      <collision>
+	<geometry>
+          <mesh filename="package://schunk_svh_driver/description/meshes/f11.dae" />
+	</geometry>
+      </collision>
     </link>
     <link name="${name}_p">
@@ -148,4 +198,9 @@
 	</geometry>
       </visual>
+      <collision>
+	<geometry>
+          <mesh filename="package://schunk_svh_driver/description/meshes/f12.dae" />
+	</geometry>
+      </collision>
     </link>
     <link name="${name}_t">
@@ -155,4 +210,9 @@
 	</geometry>
       </visual>
+      <collision>
+	<geometry>
+          <mesh filename="package://schunk_svh_driver/description/meshes/f13.dae" />
+	</geometry>
+      </collision>
     </link>
     <!-- MIDDLE FINGER LINKS -->
@@ -164,4 +224,10 @@
 	</geometry>
       </visual>
+      <collision>
+	<origin xyz="0 0 0.01321" />
+	<geometry>
+          <mesh filename="package://schunk_svh_driver/description/meshes/f20.dae" />
+	</geometry>
+      </collision>
     </link>
     <link name="${name}_k">
@@ -171,4 +237,9 @@
 	</geometry>
       </visual>
+      <collision>
+	<geometry>
+          <mesh filename="package://schunk_svh_driver/description/meshes/f21.dae" />
+	</geometry>
+      </collision>
     </link>
     <link name="${name}_o">
@@ -178,4 +249,9 @@
 	</geometry>
       </visual>
+      <collision>
+	<geometry>
+          <mesh filename="package://schunk_svh_driver/description/meshes/f22.dae" />
+	</geometry>
+      </collision>
     </link>
     <link name="${name}_s">
@@ -185,4 +261,9 @@
 	</geometry>
       </visual>
+      <collision>
+	<geometry>
+          <mesh filename="package://schunk_svh_driver/description/meshes/f23.dae" />
+	</geometry>
+      </collision>
     </link>
     <!-- RING FINGER LINKS -->
@@ -194,4 +275,10 @@
 	</geometry>
       </visual>
+      <collision>
+	<origin xyz="0 0 -0.01321" />
+	<geometry>
+          <mesh filename="package://schunk_svh_driver/description/meshes/f30.dae" />
+	</geometry>
+      </collision>
     </link>
     <link name="${name}_j">
@@ -201,4 +288,9 @@
 	</geometry>
       </visual>
+      <collision>
+	<geometry>
+          <mesh filename="package://schunk_svh_driver/description/meshes/f31.dae" />
+	</geometry>
+      </collision>
     </link>
     <link name="${name}_n">
@@ -208,4 +300,9 @@
 	</geometry>
       </visual>
+      <collision>
+	<geometry>
+          <mesh filename="package://schunk_svh_driver/description/meshes/f32.dae" />
+	</geometry>
+      </collision>
     </link>
     <link name="${name}_r">
@@ -215,4 +312,9 @@
 	</geometry>
       </visual>
+      <collision>
+	<geometry>
+          <mesh filename="package://schunk_svh_driver/description/meshes/f33.dae" />
+	</geometry>
+      </collision>
     </link>
     <!-- LITTLE FINGER LINKS -->
@@ -224,4 +326,10 @@
 	</geometry>
       </visual>
+      <collision>
+	<origin xyz="0 0 -0.01321" />
+	<geometry>
+          <mesh filename="package://schunk_svh_driver/description/meshes/f40.dae" />
+	</geometry>
+      </collision>
     </link>
     <link name="${name}_i">
@@ -231,4 +339,9 @@
 	</geometry>
       </visual>
+      <collision>
+	<geometry>
+          <mesh filename="package://schunk_svh_driver/description/meshes/f41.dae" />
+	</geometry>
+      </collision>
     </link>
     <link name="${name}_m">
@@ -238,4 +351,9 @@
 	</geometry>
       </visual>
+      <collision>
+	<geometry>
+          <mesh filename="package://schunk_svh_driver/description/meshes/f42.dae" />
+	</geometry>
+      </collision>
     </link>
     <link name="${name}_q">
@@ -245,4 +363,9 @@
 	</geometry>
       </visual>
+      <collision>
+	<geometry>
+          <mesh filename="package://schunk_svh_driver/description/meshes/f43.dae" />
+	</geometry>
+      </collision>
     </link>
     <joint name="${name}_Thumb_Flexion" type="revolute">
